Commit message: Switch to generating combined sdf

File: combined_human_pr2.xacro (robot description, xacro)
@@ -1,4 +1,4 @@
 <sdf version="1.5">
-  <model name="combined_human_pr2">
+  <model name="combined_human_pr2" xmlns:xacro="http://www.ros.org/wiki/xacro">
     <link name="base_footprint">
       <pose>0.0 0.0 0.0 0.0 -0.0 0.0</pose>
@@ -4542,624 +4542,10 @@
     </gripper>
     <!-- Human -->
-    <link name="trunk">
-      <pose>0.769877 -0.187804 1.031 0.0 0.0 0.0</pose><!-- Height of leg + thigh + 0.5 * trunk-->
-      <inertial>
-        <mass>37.0762</mass>
-        <pose>0.0 0.0 0.0 0.0 0.0 0.0</pose><!-- Link mass is centered -->
-        <inertia>
-          <ixx>1.674614776</ixx>
-          <iyy>0.01679029</iyy>
-          <izz>1.674614776</izz>
-          <ixy>0.0</ixy>
-          <ixz>0.0</ixz>
-          <iyz>0.0</iyz>
-        </inertia>
-      </inertial>
-      <collision name="collision">
-        <geometry>
-          <cylinder>
-            <length>0.376</length>
-            <radius>0.02</radius>
-          </cylinder>
-        </geometry>
-       </collision>
-       <visual name="visual">
-         <geometry>
-          <cylinder>
-            <length>0.376</length>
-            <radius>0.02</radius>
-          </cylinder>
-        </geometry>
-       </visual>
-    </link>
-    <link name="left_foot">
-      <pose>0.810877 -0.273304 0.0 0.0 1.570796327 0.0</pose><!-- Move forward by half length of foot. Y coordinate is half the pelvic width. Rotate to horizontal plane -->
-      <inertial>
-        <mass>1.0817</mass>
-        <pose>0.0 0.0 0.0 0.0 0.0 0.0</pose><!-- Link mass is centered -->
-        <inertia>
-          <ixx>0.00164105</ixx>
-          <iyy>0.000227357</iyy>
-          <izz>0.00164105</izz>
-          <ixy>0.0</ixy>
-          <ixz>0.0</ixz>
-          <iyz>0.0</iyz>
-        </inertia>
-      </inertial>
-      <collision name="collision">
-        <geometry>
-          <cylinder>
-            <length>0.082</length>
-            <radius>0.02</radius>
-          </cylinder>
-        </geometry>
-        <surface>
-          <friction>
-            <ode>
-              <mu>100.0</mu>
-              <mu2>100.0</mu2>
-            </ode>
-          </friction>
-        </surface>
-       </collision>
-       <visual name="visual">
-         <geometry>
-          <cylinder>
-            <length>0.082</length>
-            <radius>0.02</radius>
-          </cylinder>
-        </geometry>
-       </visual>
-       <sensor name="left_foot_contact" type="contact">
-          <contact>
-            <collision>collision</collision>
-          </contact>
-        </sensor>
-    </link>
-    <joint name="left_ankle" type="revolute">
-      <parent>left_leg</parent>
-      <child>left_foot</child>
-      <pose>0.769877 -0.273304 0.0 0.0 1.570796327 0.0</pose>
-      <axis>
-        <xyz>0.0 1 0.0</xyz>
-      </axis>
-    </joint>
-    <link name="right_foot">
-      <pose>0.810877 -0.102304 0.0 0.0 1.570796327 0.0</pose><!-- Move forward by half length of foot. Y coordinate is half the pelvic width. Rotate to horizontal plane -->
-      <inertial>
-        <mass>1.0817</mass>
-        <pose>0.0 0.0 0.0 0.0 0.0 0.0</pose><!-- Link mass is centered -->
-        <inertia>
-          <ixx>0.00164105</ixx>
-          <iyy>0.000227357</iyy>
-          <izz>0.00164105</izz>
-          <ixy>0.0</ixy>
-          <ixz>0.0</ixz>
-          <iyz>0.0</iyz>
-        </inertia>
-      </inertial>
-      <collision name="collision">
-        <geometry>
-          <cylinder>
-            <length>0.082</length>
-            <radius>0.02</radius>
-          </cylinder>
-        </geometry>
-        <surface>
-          <friction>
-            <ode>
-              <mu>100.0</mu>
-              <mu2>100.0</mu2>
-            </ode>
-          </friction>
-        </surface>
-       </collision>
-       <visual name="visual">
-         <geometry>
-          <cylinder>
-            <length>0.082</length>
-            <radius>0.02</radius>
-          </cylinder>
-        </geometry>
-       </visual>
-       <sensor name="right_foot_contact" type="contact">
-          <contact>
-            <collision>collision</collision>
-          </contact>
-        </sensor>
-    </link>
-    <joint name="right_ankle" type="revolute">
-      <parent>right_leg</parent>
-      <child>right_foot</child>
-      <pose>0.769877 -0.102304 0.0 0.0 1.570796327 0.0</pose>
-       <axis>
-        <xyz>0.0 1 0.0</xyz>
-      </axis>
-    </joint>
-    <link name="left_leg">
-      <pose>0.769877 -0.273304 0.2045 0.0 0.0 0.0</pose><!-- Y coordinate is half the pelvic width. Z coordinate is half the leg height. -->
-      <inertial>
-        <mass>3.4689</mass>
-        <pose>0.0 0.0 0.027403 0.0 0.0 0.0</pose>
-        <inertia>
-          <ixx>0.052923954</ixx>
-          <iyy>0.000276446</iyy>
-          <izz>0.052923954</izz>
-          <ixy>0.0</ixy>
-          <ixz>0.0</ixz>
-          <iyz>0.0</iyz>
-        </inertia>
-      </inertial>
-      <collision name="collision">
-        <geometry>
-          <cylinder>
-            <length>0.409</length>
-            <radius>0.02</radius>
-          </cylinder>
-        </geometry>
-       </collision>
-       <visual name="visual">
-         <geometry>
-          <cylinder>
-            <length>0.409</length>
-            <radius>0.02</radius>
-          </cylinder>
-        </geometry>
-       </visual>
-    </link>
-    <joint name="left_knee" type="revolute">
-      <parent>left_thigh</parent>
-      <child>left_leg</child>
-      <pose>0.769877 -0.273304 0.409 0.0 0.0 0.0</pose>
-      <axis>
-        <xyz>0.0 1 0.0</xyz>
-      </axis>
-    </joint>
-    <link name="right_leg">
-      <pose>0.769877 -0.102304 0.2045 0.0 0.0 0.0</pose><!-- Y coordinate is half the pelvic width. Z coordinate is half the leg height -->
-      <inertial>
-        <mass>3.4689</mass>
-        <pose>0.0 0.0 0.027403 0.0 0.0 0.0</pose>
-        <inertia>
-          <ixx>0.052923954</ixx>
-          <iyy>0.000276446</iyy>
-          <izz>0.052923954</izz>
-          <ixy>0.0</ixy>
-          <ixz>0.0</ixz>
-          <iyz>0.0</iyz>
-        </inertia>
-      </inertial>
-      <collision name="collision">
-        <geometry>
-          <cylinder>
-            <length>0.409</length>
-            <radius>0.02</radius>
-          </cylinder>
-        </geometry>
-       </collision>
-       <visual name="visual">
-         <geometry>
-          <cylinder>
-            <length>0.409</length>
-            <radius>0.02</radius>
-          </cylinder>
-        </geometry>
-       </visual>
-    </link>
-    <joint name="right_knee" type="revolute">
-      <parent>right_thigh</parent>
-      <child>right_leg</child>
-      <pose>00.769877 -0.102304	0.409 0.0 0.0 0.0</pose>
-      <axis>
-        <xyz>0.0 1 0.0</xyz>
-      </axis>
-    </joint>
-    <link name="left_thigh">
-      <pose>0.769877 -0.273304 0.626 0.0 0.0 0.0</pose><!-- Y coordinate is half the pelvic width. X coordinate is the leg height + 0.5 * thigh height -->
-      <inertial>
-        <mass>7.46</mass>
-        <pose>0.0 0.0 0.029078 0.0 0.0 0.0</pose>
-        <inertia>
-          <ixx>0.146596409</ixx>
-          <iyy>0.001321394</iyy>
-          <izz>0.146596409</izz>
-          <ixy>0.0</ixy>
-          <ixz>0.0</ixz>
-          <iyz>0.0</iyz>
-        </inertia>
-      </inertial>
-      <collision name="collision">
-        <geometry>
-          <cylinder>
-            <length>0.434</length>
-            <radius>0.02</radius>
-          </cylinder>
-        </geometry>
-       </collision>
-       <visual name="visual">
-         <geometry>
-          <cylinder>
-            <length>0.434</length>
-            <radius>0.02</radius>
-          </cylinder>
-        </geometry>
-       </visual>
-    </link>
-    <joint name="left_hip" type="revolute">
-      <parent>transpelvic_link</parent>
-      <child>left_thigh</child>
-      <pose>0.769877 -0.273304 0.843 0.0 0.0 0.0</pose> <!-- Half thigh height -->
-      <axis>
-        <xyz>0.0 1 0.0</xyz>
-      </axis>
-    </joint>
-    <link name="right_thigh">
-      <pose>0.769877 -0.102304 0.626 0.0 0.0 0.0</pose><!-- Y coordinate is half the pelvic width. X coordinate is the leg height + 0.5 * thigh height -->
-      <inertial>
-        <mass>7.46</mass>
-        <pose>0.0 0.0 0.029078 0.0 0.0 0.0</pose>
-        <inertia>
-          <ixx>0.146596409</ixx>
-          <iyy>0.001321394</iyy>
-          <izz>0.146596409</izz>
-          <ixy>0.0</ixy>
-          <ixz>0.0</ixz>
-          <iyz>0.0</iyz>
-        </inertia>
-      </inertial>
-      <collision name="collision">
-        <geometry>
-          <cylinder>
-            <length>0.434</length>
-            <radius>0.02</radius>
-          </cylinder>
-        </geometry>
-       </collision>
-       <visual name="visual">
-         <geometry>
-          <cylinder>
-            <length>0.434</length>
-            <radius>0.02</radius>
-          </cylinder>
-        </geometry>
-       </visual>
-    </link>
-    <joint name="right_hip" type="revolute">
-      <parent>transpelvic_link</parent>
-      <child>right_thigh</child>
-      <pose>0.769877 -0.102304 0.843 0.0 0.0 0.0</pose> <!-- Half thigh height -->
-      <axis>
-        <xyz>0.0 1 0.0</xyz>
-      </axis>
-    </joint>
-    <link name="transpelvic_link">
-      <pose>0.769877 -0.187804 0.843 0.0 1.570796327 1.570796327</pose><!-- Height of leg + thigh, rotated to ground plane and rotated about the trunk -->
-      <!-- No inertial properties. Visualization only -->
-      <collision name="collision">
-        <geometry>
-          <cylinder>
-            <length>0.171</length>
-            <radius>0.02</radius>
-          </cylinder>
-        </geometry>
-       </collision>
-       <visual name="visual">
-         <geometry>
-          <cylinder>
-            <length>0.171</length>
-            <radius>0.02</radius>
-          </cylinder>
-        </geometry>
-       </visual>
-    </link>
-    <joint name="lower_spine" type="revolute">
-      <parent>trunk</parent>
-      <child>transpelvic_link</child>
-      <pose>0.769877 -0.187804 0.843 0.0 0.0 0.0</pose>
-      <axis>
-        <xyz>0.0 1 0.0</xyz>
-      </axis>
-    </joint>
-    <joint name="upper_spine" type="revolute">
-      <parent>trunk</parent>
-      <child>clavicular_link</child>
-      <pose>0.769877 -0.187804 1.219 0.0 0.0 0.0</pose>
-      <axis>
-        <xyz>0.0 1 0.0</xyz>
-      </axis>
-    </joint>
-    <link name="clavicular_link">
-      <pose>0.769877 -0.187804 1.219 0.0 1.570796327 1.570796327</pose><!-- Height of leg + thigh + trunk, rotated to ground plane and rotated about the trunk -->
-      <!-- No inertial properties. Visualization only -->
-      <collision name="collision">
-        <geometry>
-          <cylinder>
-            <length>0.163</length>
-            <radius>0.02</radius>
-          </cylinder>
-        </geometry>
-       </collision>
-       <visual name="visual">
-         <geometry>
-          <cylinder>
-            <length>0.163</length>
-            <radius>0.02</radius>
-          </cylinder>
-        </geometry>
-       </visual>
-    </link>
-    <joint name="neck" type="revolute">
-      <parent>clavicular_link</parent>
-      <child>head_neck</child>
-      <pose>0.769877 -0.187804 1.219 0.0 0.0 0.0</pose>
-      <axis>
-        <xyz>0.0 1 0.0</xyz>
-      </axis>
-    </joint>
-    <link name="head_neck">
-      <pose>0.769877 -0.187804 1.3815 0.0 0.0 0.0</pose><!-- Height of leg + thigh + trunk + 0.5 * head-neck -->
-      <inertial>
-        <mass>6.0426</mass>
-        <pose>0.0 0.0 0.1625 0.0 0.0 0.0</pose>
-        <inertia>
-          <ixx>0.156387114</ixx>
-          <iyy>0.000734459</iyy>
-          <izz>0.156387114</izz>
-          <ixy>0.0</ixy>
-          <ixz>0.0</ixz>
-          <iyz>0.0</iyz>
-        </inertia>
-      </inertial>
-      <collision name="collision">
-        <geometry>
-          <cylinder>
-            <length>0.325</length>
-            <radius>0.02</radius>
-          </cylinder>
-        </geometry>
-       </collision>
-       <visual name="visual">
-         <geometry>
-          <cylinder>
-            <length>0.325</length>
-            <radius>0.02</radius>
-          </cylinder>
-        </geometry>
-       </visual>
-    </link>
-    <link name="left_upper_arm">
-      <pose>0.769877 -0.269304 1.37 0.0 0.0 0.0</pose><!-- Y coordinate is half the pelvic width. Z coordinate is leg + thigh + trunk + 0.5 * upper arm -->
-      <inertial>
-        <mass>2.0888</mass>
-        <pose>0.0 0.0 -0.019328 0.0 0.0 0.0</pose>
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