Commit message: Lots of fixes to joints and models

File: combined_human_pr2.xacro (robot description, xacro)
@@ -39,6 +39,4 @@
         </surface>
       </collision>
-      <!-- Moby lacks mesh support -->
-      <!--
       <collision name="base_footprint_collision_base_link">
         <pose>0.0 0.0 0.051 0.0 -0.0 0.0</pose>
@@ -58,5 +56,4 @@
         </surface>
       </collision>
-      -->
       <visual name="base_footprint_visual">
         <pose>0.0 0.0 0.0 0.0 -0.0 0.0</pose>
@@ -81,6 +78,4 @@
         </material>
       </visual>
-      <!-- Moby lacks mesh support -->
-      <!--
       <visual name="base_footprint_visual_base_link">
         <pose>0.0 0.0 0.051 0.0 -0.0 0.0</pose>
@@ -92,5 +87,4 @@
         </geometry>
       </visual>
-      -->
       <velocity_decay>
         <linear>0.0</linear>
@@ -166,6 +160,4 @@
         </inertia>
       </inertial>
-      <!-- Moby lacks mesh support -->
-      <!--
       <collision name="bl_caster_rotation_link_collision">
         <pose>0.0 0.0 0.0 0.0 -0.0 0.0</pose>
@@ -185,7 +177,4 @@
         </surface>
       </collision>
-      -->
-      <!-- Moby lacks mesh support -->
-      <!--
       <visual name="bl_caster_rotation_link_visual">
         <pose>0.0 0.0 0.0 0.0 -0.0 0.0</pose>
@@ -203,5 +192,4 @@
         </material>
       </visual>
-      -->
       <gravity>1</gravity>
       <velocity_decay>
@@ -267,6 +255,4 @@
         </surface>
       </collision>
-      <!-- Moby lacks mesh support -->
-      <!--
       <visual name="bl_caster_l_wheel_link_visual">
         <pose>0.0 0.0 0.0 0.0 -0.0 0.0</pose>
@@ -278,5 +264,4 @@
         </geometry>
       </visual>
-      -->
       <gravity>1</gravity>
       <velocity_decay>
@@ -342,6 +327,4 @@
         </surface>
       </collision>
-      <!-- Moby lacks mesh support -->
-      <!--
       <visual name="bl_caster_r_wheel_link_visual">
         <pose>0.0 0.0 0.0 0.0 -0.0 0.0</pose>
@@ -353,5 +336,4 @@
         </geometry>
       </visual>
-      -->
       <gravity>1</gravity>
       <velocity_decay>
@@ -392,6 +374,4 @@
         </inertia>
       </inertial>
-      <!-- Moby lacks mesh support -->
-      <!--
       <collision name="br_caster_rotation_link_collision">
         <pose>0.0 0.0 0.0 0.0 -0.0 0.0</pose>
@@ -411,7 +391,4 @@
         </surface>
       </collision>
-      -->
-      <!-- Moby lacks mesh support -->
-      <!--
       <visual name="br_caster_rotation_link_visual">
         <pose>0.0 0.0 0.0 0.0 -0.0 0.0</pose>
@@ -429,5 +406,4 @@
         </material>
       </visual>
-      -->
       <gravity>1</gravity>
       <velocity_decay>
@@ -493,6 +469,4 @@
         </surface>
       </collision>
-      <!-- Moby lacks mesh support -->
-      <!--
       <visual name="br_caster_l_wheel_link_visual">
         <pose>0.0 0.0 0.0 0.0 -0.0 0.0</pose>
@@ -504,5 +478,4 @@
         </geometry>
       </visual>
-      -->
       <gravity>1</gravity>
       <velocity_decay>
@@ -568,6 +541,4 @@
         </surface>
       </collision>
-      <!-- Moby lacks mesh support -->
-      <!--
       <visual name="br_caster_r_wheel_link_visual">
         <pose>0.0 0.0 0.0 0.0 -0.0 0.0</pose>
@@ -579,5 +550,4 @@
         </geometry>
       </visual>
-      -->
       <gravity>1</gravity>
       <velocity_decay>
@@ -618,6 +588,4 @@
         </inertia>
       </inertial>
-      <!-- Moby lacks mesh support -->
-      <!--
       <collision name="fl_caster_rotation_link_collision">
         <pose>0.0 0.0 0.0 0.0 -0.0 0.0</pose>
@@ -637,7 +605,4 @@
         </surface>
       </collision>
-      -->
-      <!-- Moby lacks mesh support -->
-      <!--
       <visual name="fl_caster_rotation_link_visual">
         <pose>0.0 0.0 0.0 0.0 -0.0 0.0</pose>
@@ -655,5 +620,4 @@
         </material>
       </visual>
-      -->
       <gravity>1</gravity>
       <velocity_decay>
@@ -719,6 +683,4 @@
         </surface>
       </collision>
-      <!-- Moby lacks mesh support -->
-      <!--
       <visual name="fl_caster_l_wheel_link_visual">
         <pose>0.0 0.0 0.0 0.0 -0.0 0.0</pose>
@@ -730,5 +692,4 @@
         </geometry>
       </visual>
-      -->
       <gravity>1</gravity>
       <velocity_decay>
@@ -794,6 +755,4 @@
         </surface>
       </collision>
-      <!-- Moby lacks mesh support -->
-      <!--
       <visual name="fl_caster_r_wheel_link_visual">
         <pose>0.0 0.0 0.0 0.0 -0.0 0.0</pose>
@@ -805,5 +764,4 @@
         </geometry>
       </visual>
-      -->
       <gravity>1</gravity>
       <velocity_decay>
@@ -844,6 +802,4 @@
         </inertia>
       </inertial>
-      <!-- Moby lacks mesh support -->
-      <!--
       <collision name="fr_caster_rotation_link_collision">
         <pose>0.0 0.0 0.0 0.0 -0.0 0.0</pose>
@@ -863,7 +819,4 @@
         </surface>
       </collision>
-      -->
-      <!-- Moby lacks mesh support -->
-      <!--
       <visual name="fr_caster_rotation_link_visual">
         <pose>0.0 0.0 0.0 0.0 -0.0 0.0</pose>
@@ -881,5 +834,4 @@
         </material>
       </visual>
-      -->
       <gravity>1</gravity>
       <velocity_decay>
@@ -945,6 +897,4 @@
         </surface>
       </collision>
-      <!-- Moby lacks mesh support -->
-      <!--
       <visual name="fr_caster_l_wheel_link_visual">
         <pose>0.0 0.0 0.0 0.0 -0.0 0.0</pose>
@@ -956,5 +906,4 @@
         </geometry>
       </visual>
-      -->
       <gravity>1</gravity>
       <velocity_decay>
@@ -1020,6 +969,4 @@
         </surface>
       </collision>
-      <!-- Moby lacks mesh support -->
-      <!--
       <visual name="fr_caster_r_wheel_link_visual">
         <pose>0.0 0.0 0.0 0.0 -0.0 0.0</pose>
@@ -1031,5 +978,4 @@
         </geometry>
       </visual>
-      -->
       <gravity>1</gravity>
       <velocity_decay>
@@ -1070,6 +1016,4 @@
         </inertia>
       </inertial>
-      <!-- Moby lacks mesh support -->
-      <!--
       <collision name="torso_lift_link_collision">
         <pose>0.0 0.0 0.0 0.0 -0.0 0.0</pose>
@@ -1089,7 +1033,4 @@
         </surface>
       </collision>
-      -->
-      <!-- Moby lacks mesh support -->
-      <!--
       <visual name="torso_lift_link_visual">
         <pose>0.0 0.0 0.0 0.0 -0.0 0.0</pose>
@@ -1101,5 +1042,4 @@
         </geometry>
       </visual>
-      -->
       <gravity>1</gravity>
       <velocity_decay>
@@ -1155,6 +1095,4 @@
         </inertia>
       </inertial>
-      <!-- Moby lacks mesh support -->
-      <!--
       <collision name="head_pan_link_collision">
         <pose>0.0 0.0 0.0 0.0 -0.0 0.0</pose>
@@ -1175,5 +1113,4 @@
         </geometry>
       </visual>
-      -->
       <velocity_decay>
         <linear>0.0</linear>
@@ -1214,6 +1151,4 @@
         </inertia>
       </inertial>
-      <!-- Moby lacks mesh support -->
-      <!--
       <collision name="head_tilt_link_collision">
         <pose>0.0 0.0 0.0 0.0 -0.0 0.0</pose>
@@ -1225,5 +1160,4 @@
         </geometry>
       </collision>
-      -->
       <collision name="head_tilt_link_collision_head_plate_frame">
         <pose>0.0232 0.0 0.0645 0.0 -0.0 0.0</pose>
@@ -1242,6 +1176,4 @@
         </surface>
       </collision>
-      <!-- Moby lacks mesh support -->
-      <!--
       <visual name="head_tilt_link_visual">
         <pose>0.0 0.0 0.0 0.0 -0.0 0.0</pose>
@@ -1253,5 +1185,4 @@
         </geometry>
       </visual>
-      -->
       <visual name="head_tilt_link_visual_double_stereo_link">
         <pose>0.0132 0.0 0.0895 0.0 -0.0 0.0</pose>
@@ -1545,6 +1476,4 @@
         </inertia>
       </inertial>
-      <!-- Moby lacks mesh support -->
-      <!--
       <collision name="l_shoulder_pan_link_collision">
         <pose>0.0 0.0 0.0 0.0 -0.0 0.0</pose>
@@ -1564,7 +1493,4 @@
         </surface>
       </collision>
-      -->
-      <!-- Moby lacks mesh support -->
-      <!--
       <visual name="l_shoulder_pan_link_visual">
         <pose>0.0 0.0 0.0 0.0 -0.0 0.0</pose>
@@ -1576,5 +1502,4 @@
         </geometry>
       </visual>
-      -->
       <gravity>0.0</gravity>
       <velocity_decay>
@@ -1625,6 +1550,4 @@
         </inertia>
       </inertial>
-      <!-- Moby lacks mesh support -->
-      <!--
       <collision name="l_shoulder_lift_link_collision">
         <pose>0.0 0.0 0.0 0.0 -0.0 0.0</pose>
@@ -1644,7 +1567,4 @@
         </surface>
       </collision>
-      -->
-      <!-- Moby lacks mesh support -->
-      <!--
       <visual name="l_shoulder_lift_link_visual">
         <pose>0.0 0.0 0.0 0.0 -0.0 0.0</pose>
@@ -1656,5 +1576,4 @@
         </geometry>
       </visual>
-      -->
       <gravity>0.0</gravity>
       <velocity_decay>
@@ -1705,6 +1624,4 @@
         </inertia>
       </inertial>
-      <!-- Moby lacks mesh support -->
-      <!--
       <collision name="l_upper_arm_roll_link_collision">
         <pose>0.0 0.0 0.0 0.0 -0.0 0.0</pose>
@@ -1724,7 +1641,4 @@
         </surface>
       </collision>
-      -->
-      <!-- Moby lacks mesh support -->
-      <!--
       <collision name="l_upper_arm_roll_link_collision_l_upper_arm_link">
         <pose>0.0 0.0 0.0 0.0 -0.0 0.0</pose>
@@ -1752,7 +1666,4 @@
         </surface>
       </collision>
-      -->
-      <!-- Moby lacks mesh support -->
-      <!--
       <visual name="l_upper_arm_roll_link_visual">
         <pose>0.0 0.0 0.0 0.0 -0.0 0.0</pose>
@@ -1779,5 +1690,4 @@
         </geometry>
       </visual>
-      -->
       <velocity_decay>
         <linear>0.0</linear>
@@ -1833,6 +1743,4 @@
         </inertia>
       </inertial>
-      <!-- Moby lacks mesh support -->
-      <!--
       <collision name="l_elbow_flex_link_collision">
         <pose>0.0 0.0 0.0 0.0 -0.0 0.0</pose>
@@ -1852,7 +1760,4 @@
         </surface>
       </collision>
-      -->
-      <!-- Moby lacks mesh support -->
-      <!--
       <visual name="l_elbow_flex_link_visual">
         <pose>0.0 0.0 0.0 0.0 -0.0 0.0</pose>
@@ -1864,5 +1769,4 @@
         </geometry>
       </visual>
-      -->
       <gravity>0.0</gravity>
       <velocity_decay>
@@ -1913,6 +1817,4 @@
         </inertia>
       </inertial>
-      <!-- Moby lacks mesh support -->
-      <!--
       <collision name="l_forearm_roll_link_collision">
         <pose>0.0 0.0 0.0 0.0 -0.0 0.0</pose>
@@ -1932,7 +1834,4 @@
         </surface>
       </collision>
-      -->
-      <!-- Moby lacks mesh support -->
-      <!--
       <collision name="l_forearm_roll_link_collision_l_forearm_link">
         <pose>0.0 0.0 0.0 0.0 -0.0 0.0</pose>
@@ -1960,7 +1859,4 @@
         </surface>
       </collision>
-      -->
-      <!-- Moby lacks mesh support -->
-      <!--
       <visual name="l_forearm_roll_link_visual">
         <pose>0.0 0.0 0.0 0.0 -0.0 0.0</pose>
@@ -1978,7 +1874,4 @@
         </material>
       </visual>
-      -->
-      <!-- Moby lacks mesh support -->
-      <!--
       <visual name="l_forearm_roll_link_visual_l_forearm_link">
         <pose>0.0 0.0 0.0 0.0 -0.0 0.0</pose>
@@ -1990,5 +1883,4 @@
         </geometry>
       </visual>
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
File: human-model-include.xacro (robot description, xacro)
@@ -77,7 +77,7 @@
     </link>
     <joint name='${prefix}left_ankle' type='revolute'>
-      <parent>left_leg</parent>
-      <child>left_foot</child>
-      <pose>${0.0 + xoffset} ${-0.0855 + yoffset} ${0.0 + zoffset} 0.0 1.570796327 0.0</pose>
+      <parent>${prefix}left_leg</parent>
+      <child>${prefix}left_foot</child>
+      <pose>0.0 0.0 0.0 0.0 1.570796327 0.0</pose>
       <axis>
         <xyz>0.0 1 0.0</xyz>
@@ -129,7 +129,7 @@
     </link>
     <joint name='${prefix}right_ankle' type='revolute'>
-      <parent>right_leg</parent>
-      <child>right_foot</child>
-      <pose>${0.0 + xoffset} ${0.0855 + yoffset} ${0.0 + zoffset} 0.0 1.570796327 0.0</pose>
+      <parent>${prefix}right_leg</parent>
+      <child>${prefix}right_foot</child>
+      <pose>0.0 0.0 0.0 0.0 1.570796327 0.0</pose>
        <axis>
         <xyz>0.0 1 0.0</xyz>
@@ -168,7 +168,7 @@
     </link>
     <joint name='${prefix}left_knee' type='revolute'>
-      <parent>left_thigh</parent>
-      <child>left_leg</child>
-      <pose>${0.0 + xoffset} ${-0.0855 + yoffset} ${0.409 + zoffset} 0.0 0.0 0.0</pose>
+      <parent>${prefix}left_thigh</parent>
+      <child>${prefix}left_leg</child>
+      <pose>0.0 0.0 0.2045 0.0 0.0 0.0</pose>
       <axis>
         <xyz>0.0 1 0.0</xyz>
@@ -207,7 +207,7 @@
     </link>
     <joint name='${prefix}right_knee' type='revolute'>
-      <parent>right_thigh</parent>
-      <child>right_leg</child>
-      <pose>${0.0 + xoffset} ${0.0855 + yoffset} ${0.409 + zoffset} 0.0 0.0 0.0</pose>
+      <parent>${prefix}right_thigh</parent>
+      <child>${prefix}right_leg</child>
+      <pose>0.0 0.0 0.2045 0.0 0.0 0.0</pose>
       <axis>
         <xyz>0.0 1 0.0</xyz>
@@ -246,7 +246,7 @@
     </link>
     <joint name='${prefix}left_hip' type='revolute'>
-      <parent>transpelvic_link</parent>
-      <child>left_thigh</child>
-      <pose>${0.0 + xoffset} ${-0.0855 + yoffset} ${0.843 + zoffset} 0.0 0.0 0.0</pose> <!--Height leg + thigh -->
+      <parent>${prefix}transpelvic_link</parent>
+      <child>${prefix}left_thigh</child>
+      <pose>0.0 0.0 0.217 0.0 0.0 0.0</pose> <!--Height leg + thigh -->
       <axis>
         <xyz>0.0 1 0.0</xyz>
@@ -285,7 +285,7 @@
     </link>
     <joint name='${prefix}right_hip' type='revolute'>
-      <parent>transpelvic_link</parent>
-      <child>right_thigh</child>
-      <pose>${0.0 + xoffset} ${0.0855 + yoffset} ${0.843 + zoffset} 0.0 0.0 0.0</pose> <!-- leg + thigh height -->
+      <parent>${prefix}transpelvic_link</parent>
+      <child>${prefix}right_thigh</child>
+      <pose>0.0 0.0 0.217 0.0 0.0 0.0</pose> <!-- leg + thigh height -->
       <axis>
         <xyz>0.0 1 0.0</xyz>
@@ -313,7 +313,7 @@
     </link>
     <joint name='${prefix}lower_spine' type='revolute'>
-      <parent>trunk</parent>
-      <child>transpelvic_link</child>
-      <pose>${0.0 + xoffset} ${0.0 + yoffset} ${0.843 + zoffset} 0.0 0.0 0.0</pose>
+      <parent>${prefix}trunk</parent>
+      <child>${prefix}transpelvic_link</child>
+      <pose>0.0 0.0 0.0 0.0 0.0 0.0</pose>
       <axis>
         <xyz>0.0 1 0.0</xyz>
@@ -321,7 +321,7 @@
     </joint>
     <joint name='${prefix}upper_spine' type='revolute'>
-      <parent>trunk</parent>
-      <child>clavicular_link</child>
-      <pose>${0.0 + xoffset} ${0.0 + yoffset} ${1.219 + zoffset} 0.0 0.0 0.0</pose>
+      <parent>${prefix}trunk</parent>
+      <child>${prefix}clavicular_link</child>
+      <pose>0.0 0.0 0.0 0.0 0.0 0.0</pose>
       <axis>
         <xyz>0.0 1 0.0</xyz>
@@ -349,7 +349,7 @@
     </link>
     <joint name='${prefix}neck' type='revolute'>
-      <parent>clavicular_link</parent>
-      <child>head_neck</child>
-      <pose>${0.0 + xoffset} ${0.0 + yoffset} ${1.219 + zoffset} 0.0 0.0 0.0</pose>
+      <parent>${prefix}clavicular_link</parent>
+      <child>${prefix}head_neck</child>
+      <pose>0.0 0.0 -0.1625 0.0 0.0 0.0</pose>
       <axis>
         <xyz>0.0 1 0.0</xyz>
@@ -419,7 +419,7 @@
     </link>
     <joint name='${prefix}left_shoulder' type='revolute'>
-      <parent>clavicular_link</parent>
-      <child>left_upper_arm</child>
-      <pose>${0.0 + xoffset} ${-0.0815 + yoffset} ${1.219 + zoffset} 0.0 0.0 0.0</pose>
+      <parent>${prefix}clavicular_link</parent>
+      <child>${prefix}left_upper_arm</child>
+      <pose>0.0 0.0 -0.151 0.0 0.0 0.0</pose>
       <axis>
         <xyz>0.0 1 0.0</xyz>
@@ -458,7 +458,7 @@
     </link>
     <joint name='${prefix}right_shoulder' type='revolute'>
-      <parent>clavicular_link</parent>
-      <child>right_upper_arm</child>
-      <pose>${0.0 + xoffset} ${0.0815 + yoffset} ${1.219 + zoffset} 0.0 0.0 0.0</pose>
+      <parent>${prefix}clavicular_link</parent>
+      <child>${prefix}right_upper_arm</child>
+      <pose>0.0 0.0 -0.151 0.0 0.0 0.0</pose>
       <axis>
         <xyz>0.0 1 0.0</xyz>
@@ -497,7 +497,7 @@
     </link>
     <joint name='${prefix}left_elbow' type='revolute'>
-      <parent>left_upper_arm</parent>
-      <child>left_forearm</child>
-      <pose>${0.0 + xoffset} ${-0.0815 + yoffset} ${1.521 + zoffset} 0.0 0.0 0.0</pose>
+      <parent>${prefix}left_upper_arm</parent>
+      <child>${prefix}left_forearm</child>
+      <pose>0.0 0.0 -0.136 0.0 0.0 0.0</pose>
       <axis>
         <xyz>0.0 1 0.0</xyz>
@@ -536,7 +536,7 @@
     </link>
     <joint name='${prefix}right_elbow' type='revolute'>
-      <parent>right_upper_arm</parent>
-      <child>right_forearm</child>
-      <pose>${0.0 + xoffset} ${0.0815 + yoffset} ${1.521 + zoffset} 0.0 0.0 0.0</pose>
+      <parent>${prefix}right_upper_arm</parent>
+      <child>${prefix}right_forearm</child>
+      <pose>0.0 0.0 -0.136 0.0 0.0 0.0</pose>
       <axis>
         <xyz>0.0 1 0.0</xyz>
@@ -575,7 +575,7 @@
     </link>
     <joint name='${prefix}left_wrist' type='revolute'>
-      <parent>left_forearm</parent>
-      <child>left_hand</child>
-      <pose>${0.0 + xoffset} ${-0.0815 + yoffset} ${1.793 + zoffset} 0.0 0.0 0.0</pose>
+      <parent>${prefix}left_forearm</parent>
+      <child>${prefix}left_hand</child>
+      <pose>0.0 0.0 -0.035 0.0 0.0 0.0</pose>
       <axis>
         <xyz>0.0 1 0.0</xyz>
@@ -614,7 +614,7 @@
     </link>
     <joint name='${prefix}right_wrist' type='revolute'>
-      <parent>right_forearm</parent>
-      <child>right_hand</child>
-      <pose>${0.0 + xoffset} ${0.0815 + yoffset} ${1.793 + zoffset} 0.0 0.0 0.0</pose>
+      <parent>${prefix}right_forearm</parent>
+      <child>${prefix}right_hand</child>
+      <pose>0.0 0.0 -0.035 0.0 0.0 0.0</pose>
       <axis>
         <xyz>0.0 1 0.0</xyz>

Commit message: Adjust gripper position on human to left hip

File: combined_human_pr2.xacro (robot description, xacro)
@@ -4302,6 +4302,6 @@
     <!-- Human -->
     <!-- TODO: These should not be needed but parameters aren"t working -->
-    <xacro:property name="xoffset" value="0.769877" />
-    <xacro:property name="yoffset" value="-0.187804" />
+    <xacro:property name="xoffset" value="0.939280" />
+    <xacro:property name="yoffset" value="-0.25" />
     <xacro:property name="zoffset" value="0" />
     <xacro:property name="prefix" value="human_" />
