Commit message: Working PR2 that attempts to hold up the human

File: combined_human_pr2.xacro (robot description, xacro)
@@ -1,4310 +1,9 @@
 <sdf version="1.5">
   <model name="combined_human_pr2" xmlns:xacro="http://www.ros.org/wiki/xacro">
-    <link name="base_footprint">
-      <pose>0.0 0.0 0.0 0.0 -0.0 0.0</pose>
-      <inertial>
-        <pose>-0.0624209 0.0 0.201365 0.0 -0.0 0.0</pose>
-        <mass>118.001</mass>
-        <inertia>
-          <ixx>6.13665</ixx>
-          <ixy>-0.00971993</ixy>
-          <ixz>1.455</ixz>
-          <iyy>6.20983</iyy>
-          <iyz>-0.00737958</iyz>
-          <izz>3.75933</izz>
-        </inertia>
-      </inertial>
-      <collision name="base_footprint_collision">
-        <pose>0.0 0.0 0.071 0.0 -0.0 0.0</pose>
-        <geometry>
-          <box>
-            <size>0.001 0.001 0.001</size>
-          </box>
-        </geometry>
-      </collision>
-      <collision name="base_footprint_collision_base_bellow_link">
-        <pose>-0.29 0.0 0.851 0.0 -0.0 0.0</pose>
-        <geometry>
-          <box>
-            <size>0.05 0.37 0.3</size>
-          </box>
-        </geometry>
-        <surface>
-          <contact>
-            <ode/>
-          </contact>
-          <friction>
-            <ode/>
-          </friction>
-        </surface>
-      </collision>
-      <collision name="base_footprint_collision_base_link">
-        <pose>0.0 0.0 0.051 0.0 -0.0 0.0</pose>
-        <geometry>
-          <mesh>
-            <scale>1 1 1</scale>
-            <uri>/Users/joshualurz/.gazebo/models/pr2/pr2_description/meshes/base_v0/base_L.stl</uri>
-          </mesh>
-        </geometry>
-        <surface>
-          <contact>
-            <ode/>
-          </contact>
-          <friction>
-            <ode/>
-          </friction>
-        </surface>
-      </collision>
-      <visual name="base_footprint_visual">
-        <pose>0.0 0.0 0.0 0.0 -0.0 0.0</pose>
-        <geometry>
-          <box>
-            <size>0.01 0.01 0.01</size>
-          </box>
-        </geometry>
-      </visual>
-      <visual name="base_footprint_visual_base_bellow_link">
-        <pose>-0.29 0.0 0.851 0.0 -0.0 0.0</pose>
-        <geometry>
-          <box>
-            <size>0.05 0.37 0.3</size>
-          </box>
-        </geometry>
-        <material>
-          <script>
-            <name>PR2/Black</name>
-            <uri>__default__</uri>
-          </script>
-        </material>
-      </visual>
-      <visual name="base_footprint_visual_base_link">
-        <pose>0.0 0.0 0.051 0.0 -0.0 0.0</pose>
-        <geometry>
-          <mesh>
-            <scale>1 1 1</scale>
-            <uri>/Users/joshualurz/.gazebo/models/pr2/pr2_description/meshes/base_v0/base.dae</uri>
-          </mesh>
-        </geometry>
-      </visual>
-      <velocity_decay>
-        <linear>0.0</linear>
-        <angular>0.0</angular>
-      </velocity_decay>
-      <sensor name="base_contact_sensor" type="contact">
-        <always_on>1</always_on>
-        <update_rate>100.0</update_rate>
-        <contact>
-          <collision>base_link_geom</collision>
-          <topic>__default_topic__</topic>
-        </contact>
-        <!-- <plugin name="base_gazebo_ros_bumper_controller" filename="libgazebo_ros_bumper.so">
-          <alwaysOn>true</alwaysOn>
-          <updateRate>100.0.0</updateRate>
-          <bumperTopicName>base_bumper</bumperTopicName>
-          <frameName>world</frameName>
-        </plugin> -->
-        <pose>0.0 0.0 0.051 0.0 -0.0 0.0</pose>
-      </sensor>
-      <velocity_decay>
-        <linear>0.0</linear>
-        <angular>0.0</angular>
-      </velocity_decay>
-      <gravity>1</gravity>
-      <velocity_decay>
-        <linear>0.0</linear>
-        <angular>0.0</angular>
-      </velocity_decay>
-      <self_collide>0.0</self_collide>
-      <sensor name="base_laser" type="ray">
-        <always_on>1</always_on>
-        <update_rate>20.0</update_rate>
-        <visualize>0.0</visualize>
-        <ray>
-          <scan>
-            <horizontal>
-              <samples>640.0</samples>
-              <resolution>1</resolution>
-              <min_angle>-2.2689</min_angle>
-              <max_angle>2.2689</max_angle>
-            </horizontal>
-          </scan>
-          <range>
-            <min>0.08</min>
-            <max>10.0</max>
-            <resolution>0.01</resolution>
-          </range>
-        </ray>
-        <!-- <plugin name="gazebo_ros_base_laser_controller" filename="libgazebo_ros_laser.so">
-          <gaussianNoise>0.005</gaussianNoise>
-          <alwaysOn>true</alwaysOn>
-          <updateRate>20.0</updateRate>
-          <topicName>base_scan</topicName>
-          <frameName>base_laser_link</frameName>
-          <hokuyoMinIntensity>101</hokuyoMinIntensity>
-        </plugin> -->
-        <pose>0.275 0.0 0.303 0.0 -0.0 0.0</pose>
-      </sensor>
-    </link>
-    <link name="bl_caster_rotation_link">
-      <pose>-0.2246 0.2246 0.0792 0.0 -0.0 0.0</pose>
-      <inertial>
-        <pose>0.0 0.0 0.07 0.0 -0.0 0.0</pose>
-        <mass>3.47308</mass>
-        <inertia>
-          <ixx>0.0124118</ixx>
-          <ixy>-0.000711734</ixy>
-          <ixz>0.00050273</ixz>
-          <iyy>0.0152182</iyy>
-          <iyz>-4.27347e-06</iyz>
-          <izz>0.011764</izz>
-        </inertia>
-      </inertial>
-      <collision name="bl_caster_rotation_link_collision">
-        <pose>0.0 0.0 0.0 0.0 -0.0 0.0</pose>
-        <geometry>
-          <mesh>
-            <scale>1 1 1</scale>
-            <uri>/Users/joshualurz/.gazebo/models/pr2/pr2_description/meshes/base_v0/caster_L.stl</uri>
-          </mesh>
-        </geometry>
-        <surface>
-          <contact>
-            <ode/>
-          </contact>
-          <friction>
-            <ode/>
-          </friction>
-        </surface>
-      </collision>
-      <visual name="bl_caster_rotation_link_visual">
-        <pose>0.0 0.0 0.0 0.0 -0.0 0.0</pose>
-        <geometry>
-          <mesh>
-            <scale>1 1 1</scale>
-            <uri>/Users/joshualurz/.gazebo/models/pr2/pr2_description/meshes/base_v0/caster.stl</uri>
-          </mesh>
-        </geometry>
-        <material>
-          <script>
-            <name>PR2/caster_texture</name>
-            <uri>__default__</uri>
-          </script>
-        </material>
-      </visual>
-      <gravity>1</gravity>
-      <velocity_decay>
-        <linear>0.0</linear>
-        <angular>0.0</angular>
-      </velocity_decay>
-      <self_collide>0.0</self_collide>
-    </link>
-    <joint name="bl_caster_rotation_joint" type="revolute">
-      <child>bl_caster_rotation_link</child>
-      <parent>base_footprint</parent>
-      <axis>
-        <xyz>0.0 0.0 1</xyz>
-        <limit>
-          <lower>-1e+16</lower>
-          <upper>1e+16</upper>
-        </limit>
-        <dynamics>
-          <damping>1</damping>
-          <spring_reference>0.0</spring_reference>
-          <spring_stiffness>0.0</spring_stiffness>
-        </dynamics>
-        <use_parent_model_frame>1</use_parent_model_frame>
-      </axis>
-    </joint>
-    <link name="bl_caster_l_wheel_link">
-      <pose>-0.2246 0.2736 0.0792 0.0 -0.0 0.0</pose>
-      <inertial>
-        <pose>0.0 0.0 0.0 0.0 -0.0 0.0</pose>
-        <mass>0.44036</mass>
-        <inertia>
-          <ixx>0.0124118</ixx>
-          <ixy>-0.000711734</ixy>
-          <ixz>0.00050273</ixz>
-          <iyy>0.0152182</iyy>
-          <iyz>-4.27347e-06</iyz>
-          <izz>0.011764</izz>
-        </inertia>
-      </inertial>
-      <collision name="bl_caster_l_wheel_link_collision">
-        <pose>0.0 0.0 0.0 1.5708 -0.0 0.0</pose>
-        <geometry>
-          <cylinder>
-            <length>0.034</length>
-            <radius>0.074792</radius>
-          </cylinder>
-        </geometry>
-        <surface>
-          <contact>
-            <ode>
-              <kp>1e+06</kp>
-              <kd>1</kd>
-              <max_vel>100.0</max_vel>
-              <min_depth>0.0</min_depth>
-            </ode>
-          </contact>
-          <friction>
-            <ode>
-              <mu>100.0</mu>
-              <mu2>100.0</mu2>
-            </ode>
-          </friction>
-        </surface>
-      </collision>
-      <visual name="bl_caster_l_wheel_link_visual">
-        <pose>0.0 0.0 0.0 0.0 -0.0 0.0</pose>
-        <geometry>
-          <mesh>
-            <scale>1 1 1</scale>
-            <uri>/Users/joshualurz/.gazebo/models/pr2/pr2_description/meshes/base_v0/wheel.dae</uri>
-          </mesh>
-        </geometry>
-      </visual>
-      <gravity>1</gravity>
-      <velocity_decay>
-        <linear>0.0</linear>
-        <angular>0.0</angular>
-      </velocity_decay>
-      <self_collide>0.0</self_collide>
-    </link>
-    <joint name="bl_caster_l_wheel_joint" type="revolute">
-      <child>bl_caster_l_wheel_link</child>
-      <parent>bl_caster_rotation_link</parent>
-      <axis>
-        <xyz>0.0 1 0.0</xyz>
-        <limit>
-          <lower>-1e+16</lower>
-          <upper>1e+16</upper>
-        </limit>
-        <dynamics>
-          <damping>1</damping>
-          <spring_reference>0.0</spring_reference>
-          <spring_stiffness>0.0</spring_stiffness>
-        </dynamics>
-        <use_parent_model_frame>1</use_parent_model_frame>
-      </axis>
-    </joint>
-    <link name="bl_caster_r_wheel_link">
-      <pose>-0.2246 0.1756 0.0792 0.0 -0.0 0.0</pose>
-      <inertial>
-        <pose>0.0 0.0 0.0 0.0 -0.0 0.0</pose>
-        <mass>0.44036</mass>
-        <inertia>
-          <ixx>0.0124118</ixx>
-          <ixy>-0.000711734</ixy>
-          <ixz>0.00050273</ixz>
-          <iyy>0.0152182</iyy>
-          <iyz>-4.27347e-06</iyz>
-          <izz>0.011764</izz>
-        </inertia>
-      </inertial>
-      <collision name="bl_caster_r_wheel_link_collision">
-        <pose>0.0 0.0 0.0 1.5708 -0.0 0.0</pose>
-        <geometry>
-          <cylinder>
-            <length>0.034</length>
-            <radius>0.074792</radius>
-          </cylinder>
-        </geometry>
-        <surface>
-          <contact>
-            <ode>
-              <kp>1e+06</kp>
-              <kd>1</kd>
-              <max_vel>100.0</max_vel>
-              <min_depth>0.0</min_depth>
-            </ode>
-          </contact>
-          <friction>
-            <ode>
-              <mu>100.0</mu>
-              <mu2>100.0</mu2>
-            </ode>
-          </friction>
-        </surface>
-      </collision>
-      <visual name="bl_caster_r_wheel_link_visual">
-        <pose>0.0 0.0 0.0 0.0 -0.0 0.0</pose>
-        <geometry>
-          <mesh>
-            <scale>1 1 1</scale>
-            <uri>/Users/joshualurz/.gazebo/models/pr2/pr2_description/meshes/base_v0/wheel.dae</uri>
-          </mesh>
-        </geometry>
-      </visual>
-      <gravity>1</gravity>
-      <velocity_decay>
-        <linear>0.0</linear>
-        <angular>0.0</angular>
-      </velocity_decay>
-      <self_collide>0.0</self_collide>
-    </link>
-    <joint name="bl_caster_r_wheel_joint" type="revolute">
-      <child>bl_caster_r_wheel_link</child>
-      <parent>bl_caster_rotation_link</parent>
-      <axis>
-        <xyz>0.0 1 0.0</xyz>
-        <limit>
-          <lower>-1e+16</lower>
-          <upper>1e+16</upper>
-        </limit>
-        <dynamics>
-          <damping>1</damping>
-          <spring_reference>0.0</spring_reference>
-          <spring_stiffness>0.0</spring_stiffness>
-        </dynamics>
-        <use_parent_model_frame>1</use_parent_model_frame>
-      </axis>
-    </joint>
-    <link name="br_caster_rotation_link">
-      <pose>-0.2246 -0.2246 0.0792 0.0 -0.0 0.0</pose>
-      <inertial>
-        <pose>0.0 0.0 0.07 0.0 -0.0 0.0</pose>
-        <mass>3.47308</mass>
-        <inertia>
-          <ixx>0.0124118</ixx>
-          <ixy>-0.000711734</ixy>
-          <ixz>0.00050273</ixz>
-          <iyy>0.0152182</iyy>
-          <iyz>-4.27347e-06</iyz>
-          <izz>0.011764</izz>
-        </inertia>
-      </inertial>
-      <collision name="br_caster_rotation_link_collision">
-        <pose>0.0 0.0 0.0 0.0 -0.0 0.0</pose>
-        <geometry>
-          <mesh>
-            <scale>1 1 1</scale>
-            <uri>/Users/joshualurz/.gazebo/models/pr2/pr2_description/meshes/base_v0/caster_L.stl</uri>
-          </mesh>
-        </geometry>
-        <surface>
-          <contact>
-            <ode/>
-          </contact>
-          <friction>
-            <ode/>
-          </friction>
-        </surface>
-      </collision>
-      <visual name="br_caster_rotation_link_visual">
-        <pose>0.0 0.0 0.0 0.0 -0.0 0.0</pose>
-        <geometry>
-          <mesh>
-            <scale>1 1 1</scale>
-            <uri>/Users/joshualurz/.gazebo/models/pr2/pr2_description/meshes/base_v0/caster.stl</uri>
-          </mesh>
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
Commit message: Make effort configurable for the arm via xacro

File: combined_human_pr2.xacro (robot description, xacro)
@@ -1,7 +1,9 @@
 <sdf version="1.5">
   <model name="combined_human_pr2" xmlns:xacro="http://www.ros.org/wiki/xacro">
-    <xacro:include filename="pr2.nomodel.sdf" />
+   <xacro:property name="armEffort" value="0" /> <!-- Standard value is 30 -->
+    <xacro:property name="wristEffort" value="0" /> <!-- Standard value is 10 -->
+    <xacro:include filename="pr2-include.xacro" />
     <!-- Controller for the pr2 arm -->
-    <plugin name="pr2_arm_controller" filename="libStableControllerPlugin.dylib">    </plugin>
+    <!-- <plugin name="pr2_arm_controller" filename="libStableControllerPlugin.dylib">    </plugin>-->
     <!-- Human -->
     <!-- TODO: These should not be needed but parameters aren't working -->

File: pr2-include.xacro (robot description, xacro)
@@ -2754,5 +2754,5 @@
           <lower>-2.2854</lower>
           <upper>0.714602</upper>
-          <effort>30</effort>
+          <effort>${armEffort}</effort>
           <velocity>2.088</velocity>
         </limit>
@@ -2828,5 +2828,5 @@
           <lower>-0.5236</lower>
           <upper>1.3963</upper>
-          <effort>30</effort>
+          <effort>${armEffort}</effort>
           <velocity>2.082</velocity>
         </limit>
@@ -2946,5 +2946,5 @@
           <lower>-3.9</lower>
           <upper>0.8</upper>
-          <effort>30</effort>
+          <effort>${armEffort}</effort>
           <velocity>3.27</velocity>
         </limit>
@@ -3021,5 +3021,5 @@
           <lower>-2.3213</lower>
           <upper>0</upper>
-          <effort>30</effort>
+          <effort>${armEffort}</effort>
           <velocity>3.3</velocity>
         </limit>
@@ -3251,5 +3251,5 @@
           <lower>-2.18</lower>
           <upper>0</upper>
-          <effort>10</effort>
+          <effort>${wristEffort}</effort>
           <velocity>3.078</velocity>
         </limit>
