Commit message: Switch to generating human model

File: human-model-include.xacro (robot description, xacro)
@@ -1,8 +1,6 @@
-<?xml version="1.0"?>
-<sdf version="1.4">
-  <model name="human">
-    <static>false</static>
-    <link name="trunk">
-      <pose>0.0 0.0 1.031 0.0 0.0 0.0</pose><!-- Height of leg + thigh + 0.5 * trunk-->
+<?xml version='1.0'?>
+<xacro:macro xmlns:xacro="http://www.ros.org/wiki/xacro" name="human" params="xoffset yoffset zoffset">
+    <link name='trunk'>
+      <pose>${0.0 + xoffset} ${0.0 + yoffset} ${1.031 + zoffset} 0.0 0.0 0.0</pose><!-- Height of leg + thigh + 0.5 * trunk-->
       <inertial>
         <mass>37.0762</mass>
@@ -17,5 +15,5 @@
         </inertia>
       </inertial>
-      <collision name="collision">
+      <collision name='collision'>
         <geometry>
           <cylinder>
@@ -25,5 +23,5 @@
         </geometry>
        </collision>
-       <visual name="visual">
+       <visual name='visual'>
          <geometry>
           <cylinder>
@@ -34,6 +32,6 @@
        </visual>
     </link>
-    <link name="left_foot">
-      <pose>0.041 0.0855 0.0 0.0 1.570796327 0.0</pose><!-- Move forward by half length of foot. Y coordinate is half the pelvic width. Rotate to horizontal plane -->
+    <link name='left_foot'>
+      <pose>${0.041 + xoffset} ${0.0855 + yoffset} ${0.0 + zoffset} 0.0 1.570796327 0.0</pose><!-- Move forward by half length of foot. Y coordinate is half the pelvic width. Rotate to horizontal plane -->
       <inertial>
         <mass>1.0817</mass>
@@ -48,5 +46,5 @@
         </inertia>
       </inertial>
-      <collision name="collision">
+      <collision name='collision'>
         <geometry>
           <cylinder>
@@ -64,5 +62,5 @@
         </surface>
        </collision>
-       <visual name="visual">
+       <visual name='visual'>
          <geometry>
           <cylinder>
@@ -72,5 +70,5 @@
         </geometry>
        </visual>
-       <sensor name="left_foot_contact" type="contact">
+       <sensor name='left_foot_contact' type='contact'>
           <contact>
             <collision>collision</collision>
@@ -78,14 +76,14 @@
         </sensor>
     </link>
-    <joint name="left_ankle" type="revolute">
+    <joint name='left_ankle' type='revolute'>
       <parent>left_leg</parent>
       <child>left_foot</child>
-      <pose>0.0 0.0855 0.0 0.0 1.570796327 0.0</pose>
-      <axis>
-        <xyz>0.0 1 0.0</xyz>
-      </axis>
-    </joint>
-    <link name="right_foot">
-      <pose>0.041 0.0855 0.0 0.0 1.570796327 0.0</pose><!-- Move forward by half length of foot. Y coordinate is half the pelvic width. Rotate to horizontal plane -->
+      <pose>${0.0 + xoffset} ${0.0855 + yoffset} ${0.0 + zoffset} 0.0 1.570796327 0.0</pose>
+      <axis>
+        <xyz>0.0 1 0.0</xyz>
+      </axis>
+    </joint>
+    <link name='right_foot'>
+      <pose>${0.041 + xoffset} ${0.0855 + yoffset} ${0.0 + zoffset} 0.0 1.570796327 0.0</pose><!-- Move forward by half length of foot. Y coordinate is half the pelvic width. Rotate to horizontal plane -->
       <inertial>
         <mass>1.0817</mass>
@@ -100,5 +98,5 @@
         </inertia>
       </inertial>
-      <collision name="collision">
+      <collision name='collision'>
         <geometry>
           <cylinder>
@@ -116,5 +114,5 @@
         </surface>
        </collision>
-       <visual name="visual">
+       <visual name='visual'>
          <geometry>
           <cylinder>
@@ -124,5 +122,5 @@
         </geometry>
        </visual>
-       <sensor name="right_foot_contact" type="contact">
+       <sensor name='right_foot_contact' type='contact'>
           <contact>
             <collision>collision</collision>
@@ -130,14 +128,14 @@
         </sensor>
     </link>
-    <joint name="right_ankle" type="revolute">
+    <joint name='right_ankle' type='revolute'>
       <parent>right_leg</parent>
       <child>right_foot</child>
-      <pose>0.0 0.0855 0.0 0.0 1.570796327 0.0</pose>
+      <pose>${0.0 + xoffset} ${0.0855 + yoffset} ${0.0 + zoffset} 0.0 1.570796327 0.0</pose>
        <axis>
         <xyz>0.0 1 0.0</xyz>
       </axis>
     </joint>
-    <link name="left_leg">
-      <pose>0.0 0.0855 0.2045 0.0 0.0 0.0</pose><!-- Y coordinate is half the pelvic width. Z coordinate is half the leg height. -->
+    <link name='left_leg'>
+      <pose>${0.0 + xoffset} ${0.0855 + yoffset} ${0.2045 + zoffset} 0.0 0.0 0.0</pose><!-- Y coordinate is half the pelvic width. Z coordinate is half the leg height. -->
       <inertial>
         <mass>3.4689</mass>
@@ -152,5 +150,5 @@
         </inertia>
       </inertial>
-      <collision name="collision">
+      <collision name='collision'>
         <geometry>
           <cylinder>
@@ -160,5 +158,5 @@
         </geometry>
        </collision>
-       <visual name="visual">
+       <visual name='visual'>
          <geometry>
           <cylinder>
@@ -169,14 +167,14 @@
        </visual>
     </link>
-    <joint name="left_knee" type="revolute">
+    <joint name='left_knee' type='revolute'>
       <parent>left_thigh</parent>
       <child>left_leg</child>
-      <pose>0.0 0.0855 0.2045 0.0 0.0 0.0</pose>
-      <axis>
-        <xyz>0.0 1 0.0</xyz>
-      </axis>
-    </joint>
-    <link name="right_leg">
-      <pose>0.0 0.0855 0.2045 0.0 0.0 0.0</pose><!-- Y coordinate is half the pelvic width. Z coordinate is half the leg height -->
+      <pose>${0.0 + xoffset} ${0.0855 + yoffset} ${0.2045 + zoffset} 0.0 0.0 0.0</pose>
+      <axis>
+        <xyz>0.0 1 0.0</xyz>
+      </axis>
+    </joint>
+    <link name='right_leg'>
+      <pose>${0.0 + xoffset} ${0.0855 + yoffset} ${0.2045 + zoffset} 0.0 0.0 0.0</pose><!-- Y coordinate is half the pelvic width. Z coordinate is half the leg height -->
       <inertial>
         <mass>3.4689</mass>
@@ -191,5 +189,5 @@
         </inertia>
       </inertial>
-      <collision name="collision">
+      <collision name='collision'>
         <geometry>
           <cylinder>
@@ -199,5 +197,5 @@
         </geometry>
        </collision>
-       <visual name="visual">
+       <visual name='visual'>
          <geometry>
           <cylinder>
@@ -208,14 +206,14 @@
        </visual>
     </link>
-    <joint name="right_knee" type="revolute">
+    <joint name='right_knee' type='revolute'>
       <parent>right_thigh</parent>
       <child>right_leg</child>
-      <pose>0.0 0.0855 0.2045 0.0 0.0 0.0</pose>
-      <axis>
-        <xyz>0.0 1 0.0</xyz>
-      </axis>
-    </joint>
-    <link name="left_thigh">
-      <pose>0.0 0.0855 0.626 0.0 0.0 0.0</pose><!-- Y coordinate is half the pelvic width. X coordinate is the leg height + 0.5 * thigh height -->
+      <pose>${0.0 + xoffset} ${0.0855 + yoffset} ${0.2045 + zoffset} 0.0 0.0 0.0</pose>
+      <axis>
+        <xyz>0.0 1 0.0</xyz>
+      </axis>
+    </joint>
+    <link name='left_thigh'>
+      <pose>${0.0 + xoffset} ${0.0855 + yoffset} ${0.626 + zoffset} 0.0 0.0 0.0</pose><!-- Y coordinate is half the pelvic width. X coordinate is the leg height + 0.5 * thigh height -->
       <inertial>
         <mass>7.46</mass>
@@ -230,5 +228,5 @@
         </inertia>
       </inertial>
-      <collision name="collision">
+      <collision name='collision'>
         <geometry>
           <cylinder>
@@ -238,5 +236,5 @@
         </geometry>
        </collision>
-       <visual name="visual">
+       <visual name='visual'>
          <geometry>
           <cylinder>
@@ -247,14 +245,14 @@
        </visual>
     </link>
-    <joint name="left_hip" type="revolute">
+    <joint name='left_hip' type='revolute'>
       <parent>transpelvic_link</parent>
       <child>left_thigh</child>
-      <pose>0.0 0.0855 0.843 0.0 0.0 0.0</pose> <!--Height leg + thigh -->
-      <axis>
-        <xyz>0.0 1 0.0</xyz>
-      </axis>
-    </joint>
-    <link name="right_thigh">
-      <pose>0.0 0.0855 0.626 0.0 0.0 0.0</pose><!-- Y coordinate is half the pelvic width. X coordinate is the leg height + 0.5 * thigh height -->
+      <pose>${0.0 + xoffset} ${0.0855 + yoffset} ${0.843 + zoffset} 0.0 0.0 0.0</pose> <!--Height leg + thigh -->
+      <axis>
+        <xyz>0.0 1 0.0</xyz>
+      </axis>
+    </joint>
+    <link name='right_thigh'>
+      <pose>${0.0 + xoffset} ${0.0855 + yoffset} ${0.626 + zoffset} 0.0 0.0 0.0</pose><!-- Y coordinate is half the pelvic width. X coordinate is the leg height + 0.5 * thigh height -->
       <inertial>
         <mass>7.46</mass>
@@ -269,5 +267,5 @@
         </inertia>
       </inertial>
-      <collision name="collision">
+      <collision name='collision'>
         <geometry>
           <cylinder>
@@ -277,5 +275,5 @@
         </geometry>
        </collision>
-       <visual name="visual">
+       <visual name='visual'>
          <geometry>
           <cylinder>
@@ -286,16 +284,16 @@
        </visual>
     </link>
-    <joint name="right_hip" type="revolute">
+    <joint name='right_hip' type='revolute'>
       <parent>transpelvic_link</parent>
       <child>right_thigh</child>
-      <pose>0.0 0.0855 0.843 0.0 0.0 0.0</pose> <!-- leg + thigh height -->
-      <axis>
-        <xyz>0.0 1 0.0</xyz>
-      </axis>
-    </joint>
-    <link name="transpelvic_link">
-      <pose>0.0 0.0 0.843 0.0 1.570796327 1.570796327</pose><!-- Height of leg + thigh, rotated to ground plane and rotated about the trunk -->
+      <pose>${0.0 + xoffset} ${0.0855 + yoffset} ${0.843 + zoffset} 0.0 0.0 0.0</pose> <!-- leg + thigh height -->
+      <axis>
+        <xyz>0.0 1 0.0</xyz>
+      </axis>
+    </joint>
+    <link name='transpelvic_link'>
+      <pose>${0.0 + xoffset} ${0.0 + yoffset} ${0.843 + zoffset} 0.0 1.570796327 1.570796327</pose><!-- Height of leg + thigh, rotated to ground plane and rotated about the trunk -->
       <!-- No inertial properties. Visualization only -->
-      <collision name="collision">
+      <collision name='collision'>
         <geometry>
           <cylinder>
@@ -305,5 +303,5 @@
         </geometry>
        </collision>
-       <visual name="visual">
+       <visual name='visual'>
          <geometry>
           <cylinder>
@@ -314,24 +312,24 @@
        </visual>
     </link>
-    <joint name="lower_spine" type="revolute">
+    <joint name='lower_spine' type='revolute'>
       <parent>trunk</parent>
       <child>transpelvic_link</child>
-      <pose>0.0 0.0 0.843 0.0 0.0 0.0</pose>
-      <axis>
-        <xyz>0.0 1 0.0</xyz>
-      </axis>
-    </joint>
-    <joint name="upper_spine" type="revolute">
+      <pose>${0.0 + xoffset} ${0.0 + yoffset} ${0.843 + zoffset} 0.0 0.0 0.0</pose>
+      <axis>
+        <xyz>0.0 1 0.0</xyz>
+      </axis>
+    </joint>
+    <joint name='upper_spine' type='revolute'>
       <parent>trunk</parent>
       <child>clavicular_link</child>
-      <pose>0.0 0.0 1.219 0.0 0.0 0.0</pose>
-      <axis>
-        <xyz>0.0 1 0.0</xyz>
-      </axis>
-    </joint>
-    <link name="clavicular_link">
-      <pose>0.0 0.0 1.219 0.0 1.570796327 1.570796327</pose><!-- Height of leg + thigh + trunk, rotated to ground plane and rotated about the trunk -->
+      <pose>${0.0 + xoffset} ${0.0 + yoffset} ${1.219 + zoffset} 0.0 0.0 0.0</pose>
+      <axis>
+        <xyz>0.0 1 0.0</xyz>
+      </axis>
+    </joint>
+    <link name='clavicular_link'>
+      <pose>${0.0 + xoffset} ${0.0 + yoffset} ${1.219 + zoffset} 0.0 1.570796327 1.570796327</pose><!-- Height of leg + thigh + trunk, rotated to ground plane and rotated about the trunk -->
       <!-- No inertial properties. Visualization only -->
-      <collision name="collision">
+      <collision name='collision'>
         <geometry>
           <cylinder>
@@ -341,5 +339,5 @@
         </geometry>
        </collision>
-       <visual name="visual">
+       <visual name='visual'>
          <geometry>
           <cylinder>
@@ -350,14 +348,14 @@
        </visual>
     </link>
-    <joint name="neck" type="revolute">
+    <joint name='neck' type='revolute'>
       <parent>clavicular_link</parent>
       <child>head_neck</child>
-      <pose>0.0 0.0 1.219 0.0 0.0 0.0</pose>
-      <axis>
-        <xyz>0.0 1 0.0</xyz>
-      </axis>
-    </joint>
-    <link name="head_neck">
-      <pose>0.0 0.0 1.3815 0.0 0.0 0.0</pose><!-- Height of leg + thigh + trunk + 0.5 * head-neck -->
+      <pose>${0.0 + xoffset} ${0.0 + yoffset} ${1.219 + zoffset} 0.0 0.0 0.0</pose>
+      <axis>
+        <xyz>0.0 1 0.0</xyz>
+      </axis>
+    </joint>
+    <link name='head_neck'>
+      <pose>${0.0 + xoffset} ${0.0 + yoffset} ${1.3815 + zoffset} 0.0 0.0 0.0</pose><!-- Height of leg + thigh + trunk + 0.5 * head-neck -->
       <inertial>
         <mass>6.0426</mass>
@@ -372,5 +370,5 @@
         </inertia>
       </inertial>
-      <collision name="collision">
+      <collision name='collision'>
         <geometry>
           <cylinder>
@@ -380,5 +378,5 @@
         </geometry>
        </collision>
-       <visual name="visual">
+       <visual name='visual'>
          <geometry>
           <cylinder>
@@ -389,6 +387,6 @@
        </visual>
     </link>
-    <link name="left_upper_arm">
-      <pose>0.0 0.0815 1.37 0.0 0.0 0.0</pose><!-- Y coordinate is half the pelvic width. Z coordinate is leg + thigh + trunk + 0.5 * upper arm -->
+    <link name='left_upper_arm'>
+      <pose>${0.0 + xoffset} ${0.0815 + yoffset} ${1.37 + zoffset} 0.0 0.0 0.0</pose><!-- Y coordinate is half the pelvic width. Z coordinate is leg + thigh + trunk + 0.5 * upper arm -->
       <inertial>
         <mass>2.0888</mass>
@@ -403,5 +401,5 @@
         </inertia>
       </inertial>
-      <collision name="collision">
+      <collision name='collision'>
         <geometry>
           <cylinder>
@@ -411,5 +409,5 @@
         </geometry>
        </collision>
-       <visual name="visual">
+       <visual name='visual'>
          <geometry>
           <cylinder>
@@ -420,14 +418,14 @@
        </visual>
     </link>
-    <joint name="left_shoulder" type="revolute">
+    <joint name='left_shoulder' type='revolute'>
       <parent>clavicular_link</parent>
       <child>left_upper_arm</child>
-      <pose>0.0 0.0815 1.219 0.0 0.0 0.0</pose>
-      <axis>
-        <xyz>0.0 1 0.0</xyz>
-      </axis>
-    </joint>
-    <link name="right_upper_arm">
-      <pose>0.0 0.0815 1.37 0.0 0.0 0.0</pose><!-- Y coordinate is half the pelvic width. Z coordinate is leg + thigh + trunk + 0.5 * upper arm -->
+      <pose>${0.0 + xoffset} ${0.0815 + yoffset} ${1.219 + zoffset} 0.0 0.0 0.0</pose>
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