Commit message: Pre-file removal

File: human-model-include.xacro (robot description, xacro)
@@ -1,5 +1,5 @@
 <?xml version='1.0'?>
 <xacro:macro xmlns:xacro="http://www.ros.org/wiki/xacro" name="human" params="xoffset yoffset zoffset">
-    <link name='trunk'>
+    <link name='${prefix}trunk'>
       <pose>${0.0 + xoffset} ${0.0 + yoffset} ${1.031 + zoffset} 0.0 0.0 0.0</pose><!-- Height of leg + thigh + 0.5 * trunk-->
       <inertial>
@@ -32,6 +32,6 @@
        </visual>
     </link>
-    <link name='left_foot'>
-      <pose>${0.041 + xoffset} ${0.0855 + yoffset} ${0.0 + zoffset} 0.0 1.570796327 0.0</pose><!-- Move forward by half length of foot. Y coordinate is half the pelvic width. Rotate to horizontal plane -->
+    <link name='${prefix}left_foot'>
+      <pose>${0.041 + xoffset} ${-0.0855 + yoffset} ${0.0 + zoffset} 0.0 1.570796327 0.0</pose><!-- Move forward by half length of foot. Y coordinate is half the pelvic width. Rotate to horizontal plane -->
       <inertial>
         <mass>1.0817</mass>
@@ -76,13 +76,13 @@
         </sensor>
     </link>
-    <joint name='left_ankle' type='revolute'>
+    <joint name='${prefix}left_ankle' type='revolute'>
       <parent>left_leg</parent>
       <child>left_foot</child>
-      <pose>${0.0 + xoffset} ${0.0855 + yoffset} ${0.0 + zoffset} 0.0 1.570796327 0.0</pose>
-      <axis>
-        <xyz>0.0 1 0.0</xyz>
-      </axis>
-    </joint>
-    <link name='right_foot'>
+      <pose>${0.0 + xoffset} ${-0.0855 + yoffset} ${0.0 + zoffset} 0.0 1.570796327 0.0</pose>
+      <axis>
+        <xyz>0.0 1 0.0</xyz>
+      </axis>
+    </joint>
+    <link name='${prefix}right_foot'>
       <pose>${0.041 + xoffset} ${0.0855 + yoffset} ${0.0 + zoffset} 0.0 1.570796327 0.0</pose><!-- Move forward by half length of foot. Y coordinate is half the pelvic width. Rotate to horizontal plane -->
       <inertial>
@@ -128,5 +128,5 @@
         </sensor>
     </link>
-    <joint name='right_ankle' type='revolute'>
+    <joint name='${prefix}right_ankle' type='revolute'>
       <parent>right_leg</parent>
       <child>right_foot</child>
@@ -136,6 +136,6 @@
       </axis>
     </joint>
-    <link name='left_leg'>
-      <pose>${0.0 + xoffset} ${0.0855 + yoffset} ${0.2045 + zoffset} 0.0 0.0 0.0</pose><!-- Y coordinate is half the pelvic width. Z coordinate is half the leg height. -->
+    <link name='${prefix}left_leg'>
+      <pose>${0.0 + xoffset} ${-0.0855 + yoffset} ${0.2045 + zoffset} 0.0 0.0 0.0</pose><!-- Y coordinate is half the pelvic width. Z coordinate is half the leg height. -->
       <inertial>
         <mass>3.4689</mass>
@@ -167,13 +167,13 @@
        </visual>
     </link>
-    <joint name='left_knee' type='revolute'>
+    <joint name='${prefix}left_knee' type='revolute'>
       <parent>left_thigh</parent>
       <child>left_leg</child>
-      <pose>${0.0 + xoffset} ${0.0855 + yoffset} ${0.2045 + zoffset} 0.0 0.0 0.0</pose>
-      <axis>
-        <xyz>0.0 1 0.0</xyz>
-      </axis>
-    </joint>
-    <link name='right_leg'>
+      <pose>${0.0 + xoffset} ${-0.0855 + yoffset} ${0.409 + zoffset} 0.0 0.0 0.0</pose>
+      <axis>
+        <xyz>0.0 1 0.0</xyz>
+      </axis>
+    </joint>
+    <link name='${prefix}right_leg'>
       <pose>${0.0 + xoffset} ${0.0855 + yoffset} ${0.2045 + zoffset} 0.0 0.0 0.0</pose><!-- Y coordinate is half the pelvic width. Z coordinate is half the leg height -->
       <inertial>
@@ -206,14 +206,14 @@
        </visual>
     </link>
-    <joint name='right_knee' type='revolute'>
+    <joint name='${prefix}right_knee' type='revolute'>
       <parent>right_thigh</parent>
       <child>right_leg</child>
-      <pose>${0.0 + xoffset} ${0.0855 + yoffset} ${0.2045 + zoffset} 0.0 0.0 0.0</pose>
-      <axis>
-        <xyz>0.0 1 0.0</xyz>
-      </axis>
-    </joint>
-    <link name='left_thigh'>
-      <pose>${0.0 + xoffset} ${0.0855 + yoffset} ${0.626 + zoffset} 0.0 0.0 0.0</pose><!-- Y coordinate is half the pelvic width. X coordinate is the leg height + 0.5 * thigh height -->
+      <pose>${0.0 + xoffset} ${0.0855 + yoffset} ${0.409 + zoffset} 0.0 0.0 0.0</pose>
+      <axis>
+        <xyz>0.0 1 0.0</xyz>
+      </axis>
+    </joint>
+    <link name='${prefix}left_thigh'>
+      <pose>${0.0 + xoffset} ${-0.0855 + yoffset} ${0.626 + zoffset} 0.0 0.0 0.0</pose><!-- Y coordinate is half the pelvic width. X coordinate is the leg height + 0.5 * thigh height -->
       <inertial>
         <mass>7.46</mass>
@@ -245,13 +245,13 @@
        </visual>
     </link>
-    <joint name='left_hip' type='revolute'>
+    <joint name='${prefix}left_hip' type='revolute'>
       <parent>transpelvic_link</parent>
       <child>left_thigh</child>
-      <pose>${0.0 + xoffset} ${0.0855 + yoffset} ${0.843 + zoffset} 0.0 0.0 0.0</pose> <!--Height leg + thigh -->
-      <axis>
-        <xyz>0.0 1 0.0</xyz>
-      </axis>
-    </joint>
-    <link name='right_thigh'>
+      <pose>${0.0 + xoffset} ${-0.0855 + yoffset} ${0.843 + zoffset} 0.0 0.0 0.0</pose> <!--Height leg + thigh -->
+      <axis>
+        <xyz>0.0 1 0.0</xyz>
+      </axis>
+    </joint>
+    <link name='${prefix}right_thigh'>
       <pose>${0.0 + xoffset} ${0.0855 + yoffset} ${0.626 + zoffset} 0.0 0.0 0.0</pose><!-- Y coordinate is half the pelvic width. X coordinate is the leg height + 0.5 * thigh height -->
       <inertial>
@@ -284,5 +284,5 @@
        </visual>
     </link>
-    <joint name='right_hip' type='revolute'>
+    <joint name='${prefix}right_hip' type='revolute'>
       <parent>transpelvic_link</parent>
       <child>right_thigh</child>
@@ -292,5 +292,5 @@
       </axis>
     </joint>
-    <link name='transpelvic_link'>
+    <link name='${prefix}transpelvic_link'>
       <pose>${0.0 + xoffset} ${0.0 + yoffset} ${0.843 + zoffset} 0.0 1.570796327 1.570796327</pose><!-- Height of leg + thigh, rotated to ground plane and rotated about the trunk -->
       <!-- No inertial properties. Visualization only -->
@@ -312,5 +312,5 @@
        </visual>
     </link>
-    <joint name='lower_spine' type='revolute'>
+    <joint name='${prefix}lower_spine' type='revolute'>
       <parent>trunk</parent>
       <child>transpelvic_link</child>
@@ -320,5 +320,5 @@
       </axis>
     </joint>
-    <joint name='upper_spine' type='revolute'>
+    <joint name='${prefix}upper_spine' type='revolute'>
       <parent>trunk</parent>
       <child>clavicular_link</child>
@@ -328,5 +328,5 @@
       </axis>
     </joint>
-    <link name='clavicular_link'>
+    <link name='${prefix}clavicular_link'>
       <pose>${0.0 + xoffset} ${0.0 + yoffset} ${1.219 + zoffset} 0.0 1.570796327 1.570796327</pose><!-- Height of leg + thigh + trunk, rotated to ground plane and rotated about the trunk -->
       <!-- No inertial properties. Visualization only -->
@@ -348,5 +348,5 @@
        </visual>
     </link>
-    <joint name='neck' type='revolute'>
+    <joint name='${prefix}neck' type='revolute'>
       <parent>clavicular_link</parent>
       <child>head_neck</child>
@@ -356,5 +356,5 @@
       </axis>
     </joint>
-    <link name='head_neck'>
+    <link name='${prefix}head_neck'>
       <pose>${0.0 + xoffset} ${0.0 + yoffset} ${1.3815 + zoffset} 0.0 0.0 0.0</pose><!-- Height of leg + thigh + trunk + 0.5 * head-neck -->
       <inertial>
@@ -387,9 +387,9 @@
        </visual>
     </link>
-    <link name='left_upper_arm'>
-      <pose>${0.0 + xoffset} ${0.0815 + yoffset} ${1.37 + zoffset} 0.0 0.0 0.0</pose><!-- Y coordinate is half the pelvic width. Z coordinate is leg + thigh + trunk + 0.5 * upper arm -->
+    <link name='${prefix}left_upper_arm'>
+      <pose>${0.0 + xoffset} ${-0.0815 + yoffset} ${1.37 + zoffset} 0.0 0.0 0.0</pose><!-- Y coordinate is half the pelvic width. Z coordinate is leg + thigh + trunk + 0.5 * upper arm -->
       <inertial>
         <mass>2.0888</mass>
-        <pose>0.0 0.0 0.019328 0.0 0.0 0.0</pose>
+        <pose>0.0 0.0 -0.019328 0.0 0.0 0.0</pose>
         <inertia>
           <ixx>0.019752519</ixx>
@@ -418,17 +418,17 @@
        </visual>
     </link>
-    <joint name='left_shoulder' type='revolute'>
+    <joint name='${prefix}left_shoulder' type='revolute'>
       <parent>clavicular_link</parent>
       <child>left_upper_arm</child>
-      <pose>${0.0 + xoffset} ${0.0815 + yoffset} ${1.219 + zoffset} 0.0 0.0 0.0</pose>
-      <axis>
-        <xyz>0.0 1 0.0</xyz>
-      </axis>
-    </joint>
-    <link name='right_upper_arm'>
+      <pose>${0.0 + xoffset} ${-0.0815 + yoffset} ${1.219 + zoffset} 0.0 0.0 0.0</pose>
+      <axis>
+        <xyz>0.0 1 0.0</xyz>
+      </axis>
+    </joint>
+    <link name='${prefix}right_upper_arm'>
       <pose>${0.0 + xoffset} ${0.0815 + yoffset} ${1.37 + zoffset} 0.0 0.0 0.0</pose><!-- Y coordinate is half the pelvic width. Z coordinate is leg + thigh + trunk + 0.5 * upper arm -->
       <inertial>
         <mass>2.0888</mass>
-        <pose>0.0 0.0 0.019328 0.0 0.0 0.0</pose>
+        <pose>0.0 0.0 -0.019328 0.0 0.0 0.0</pose>
         <inertia>
           <ixx>0.019752519</ixx>
@@ -457,5 +457,5 @@
        </visual>
     </link>
-    <joint name='right_shoulder' type='revolute'>
+    <joint name='${prefix}right_shoulder' type='revolute'>
       <parent>clavicular_link</parent>
       <child>right_upper_arm</child>
@@ -465,9 +465,9 @@
       </axis>
     </joint>
-    <link name='left_forearm'>
-      <pose>${0.0 + xoffset} ${0.0815 + yoffset} ${1.657 + zoffset} 0.0 0.0 0.0</pose><!-- Y coordinate is half the pelvic width. Z coordinate is leg + thigh + trunk + upper arm + 0.5 * forearm -->
+    <link name='${prefix}left_forearm'>
+      <pose>${0.0 + xoffset} ${-0.0815 + yoffset} ${1.657 + zoffset} 0.0 0.0 0.0</pose><!-- Y coordinate is half the pelvic width. Z coordinate is leg + thigh + trunk + upper arm + 0.5 * forearm -->
       <inertial>
         <mass>1.1936</mass>
-        <pose>0.0 0.0 0.01904 0.0 0.0 0.0</pose>
+        <pose>0.0 0.0 -0.01904 0.0 0.0 0.0</pose>
         <inertia>
           <ixx>0.008107405</ixx>
@@ -496,17 +496,17 @@
        </visual>
     </link>
-    <joint name='left_elbow' type='revolute'>
+    <joint name='${prefix}left_elbow' type='revolute'>
       <parent>left_upper_arm</parent>
       <child>left_forearm</child>
-      <pose>${0.0 + xoffset} ${0.0815 + yoffset} ${1.521 + zoffset} 0.0 0.0 0.0</pose>
-      <axis>
-        <xyz>0.0 1 0.0</xyz>
-      </axis>
-    </joint>
-    <link name='right_forearm'>
+      <pose>${0.0 + xoffset} ${-0.0815 + yoffset} ${1.521 + zoffset} 0.0 0.0 0.0</pose>
+      <axis>
+        <xyz>0.0 1 0.0</xyz>
+      </axis>
+    </joint>
+    <link name='${prefix}right_forearm'>
       <pose>${0.0 + xoffset} ${0.0815 + yoffset} ${1.657 + zoffset} 0.0 0.0 0.0</pose><!-- Y coordinate is half the pelvic width. Z coordinate is leg + thigh + trunk + upper arm + 0.5 * forearm -->
       <inertial>
         <mass>1.1936</mass>
-        <pose>0.0 0.0 0.01904 0.0 0.0 0.0</pose>
+        <pose>0.0 0.0 -0.01904 0.0 0.0 0.0</pose>
         <inertia>
           <ixx>0.008107405</ixx>
@@ -535,5 +535,5 @@
        </visual>
     </link>
-    <joint name='right_elbow' type='revolute'>
+    <joint name='${prefix}right_elbow' type='revolute'>
       <parent>right_upper_arm</parent>
       <child>right_forearm</child>
@@ -543,6 +543,6 @@
       </axis>
     </joint>
-    <link name='left_hand'>
-      <pose>${0.0 + xoffset} ${0.0815 + yoffset} ${1.828 + zoffset} 0.0 0.0 0.0</pose><!-- Y coordinate is half the pelvic width. Z coordinate is leg + thigh + trunk + upper arm + forearm + 0.5 * hand -->
+    <link name='${prefix}left_hand'>
+      <pose>${0.0 + xoffset} ${-0.0815 + yoffset} ${1.828 + zoffset} 0.0 0.0 0.0</pose><!-- Y coordinate is half the pelvic width. Z coordinate is leg + thigh + trunk + upper arm + forearm + 0.5 * hand -->
       <inertial>
         <mass>0.4476</mass>
@@ -574,13 +574,13 @@
        </visual>
     </link>
-    <joint name='left_wrist' type='revolute'>
+    <joint name='${prefix}left_wrist' type='revolute'>
       <parent>left_forearm</parent>
       <child>left_hand</child>
-      <pose>${0.0 + xoffset} ${0.0815 + yoffset} ${1.793 + zoffset} 0.0 0.0 0.0</pose>
-      <axis>
-        <xyz>0.0 1 0.0</xyz>
-      </axis>
-    </joint>
-    <link name='right_hand'>
+      <pose>${0.0 + xoffset} ${-0.0815 + yoffset} ${1.793 + zoffset} 0.0 0.0 0.0</pose>
+      <axis>
+        <xyz>0.0 1 0.0</xyz>
+      </axis>
+    </joint>
+    <link name='${prefix}right_hand'>
       <pose>${0.0 + xoffset} ${0.0815 + yoffset} ${1.828 + zoffset} 0.0 0.0 0.0</pose><!-- Y coordinate is half the pelvic width. Z coordinate is leg + thigh + trunk + upper arm + forearm + 0.5 * hand -->
       <inertial>
@@ -613,5 +613,5 @@
        </visual>
     </link>
-    <joint name='right_wrist' type='revolute'>
+    <joint name='${prefix}right_wrist' type='revolute'>
       <parent>right_forearm</parent>
       <child>right_hand</child>

File: human-model.xacro (robot description, xacro)
@@ -6,4 +6,5 @@
     <xacro:property name="yoffset" value="0" />
     <xacro:property name="zoffset" value="0" />
+    <xacro:property name="prefix" value="" />
     <static>false</static>
     <xacro:include filename="human-model-include.xacro"/>

Commit message: Check and fix all limit values

File: human-model-include.xacro (robot description, xacro)
@@ -82,4 +82,8 @@
       <axis>
         <xyz>0.0 1 0.0</xyz>
+        <limit>
+          <lower>-0.680678408</lower>
+          <upper>0.726056969</upper>
+        </limit>
       </axis>
     </joint>
@@ -134,4 +138,8 @@
        <axis>
         <xyz>0.0 1 0.0</xyz>
+        <limit>
+          <lower>-0.680678408</lower>
+          <upper>0.726056969</upper>
+        </limit>
       </axis>
     </joint>
@@ -173,4 +181,8 @@
       <axis>
         <xyz>0.0 1 0.0</xyz>
+        <limit>
+          <lower>0</lower>
+          <upper>2.160717614</upper>
+        </limit>
       </axis>
     </joint>
@@ -212,4 +224,8 @@
       <axis>
         <xyz>0.0 1 0.0</xyz>
+        <limit>
+          <lower>0</lower>
+          <upper>2.160717614</upper>
+        </limit>
       </axis>
     </joint>
@@ -251,5 +267,16 @@
       <axis>
         <xyz>0.0 1 0.0</xyz>
-      </axis>
+        <limit>
+            <lower>-2.043780554</lower>
+            <upper>0</upper>
+        </limit>
+      </axis>
+      <axis2>
+        <xyz>0.0 0.0 -1.0</xyz>
+        <limit>
+            <lower>-0.483456203</lower>
+            <upper>1.012290966</upper>
+        </limit>
+      </axis2>
     </joint>
     <link name='${prefix}right_thigh'>
@@ -290,5 +317,16 @@
       <axis>
         <xyz>0.0 1 0.0</xyz>
-      </axis>
+        <limit>
+            <lower>-2.043780554</lower>
+            <upper>0</upper>
+        </limit>
+      </axis>
+      <axis2>
+        <xyz>0.0 0.0 1.0</xyz>
+        <limit>
+            <lower>-0.483456203</lower>
+            <upper>1.012290966</upper>
+        </limit>
+      </axis2>
     </joint>
     <link name='${prefix}transpelvic_link'>
@@ -318,4 +356,8 @@
       <axis>
         <xyz>0.0 1 0.0</xyz>
+        <limit>
+            <lower>0</lower>
+            <upper>0</upper>
+        </limit>
       </axis>
     </joint>
@@ -326,4 +368,8 @@
       <axis>
         <xyz>0.0 1 0.0</xyz>
+        <limit>
+            <lower>0</lower>
+            <upper>0</upper>
+        </limit>
       </axis>
     </joint>
@@ -354,4 +400,8 @@
       <axis>
         <xyz>0.0 1 0.0</xyz>
+        <limit>
+            <lower>0</lower>
+            <upper>0</upper>
+        </limit>
       </axis>
     </joint>
@@ -424,5 +474,16 @@
       <axis>
         <xyz>0.0 1 0.0</xyz>
-      </axis>
+        <limit>
+            <lower>3.371976115</lower>
+            <upper>-1.099557429</upper>
+        </limit>
+      </axis>
+      <axis2>
+        <xyz>0.0 0.0 -1.0</xyz>
+        <limit>
+            <lower>-2.305579942</lower>
+            <upper>0.88662726</upper>
+        </limit>
+      </axis2>
     </joint>
     <link name='${prefix}right_upper_arm'>
@@ -463,5 +524,16 @@
       <axis>
         <xyz>0.0 1 0.0</xyz>
-      </axis>
+        <limit>
+            <lower>3.371976115</lower>
+            <upper>-1.099557429</upper>
+        </limit>
+      </axis>
+      <axis2>
+        <xyz>0.0 0.0 1.0</xyz>
+        <limit>
+            <lower>-2.305579942</lower>
+            <upper>0.88662726</upper>
+        </limit>
+      </axis2>
     </joint>
     <link name='${prefix}left_forearm'>
@@ -501,5 +573,9 @@
       <pose>0.0 0.0 -0.136 0.0 0.0 0.0</pose>
       <axis>
-        <xyz>0.0 1 0.0</xyz>
+        <xyz>0.0 -1 0.0</xyz>
+        <limit>
+            <lower>0</lower>
+            <upper>2.460914245</upper>
+        </limit>
       </axis>
     </joint>
@@ -540,5 +616,9 @@
       <pose>0.0 0.0 -0.136 0.0 0.0 0.0</pose>
       <axis>
-        <xyz>0.0 1 0.0</xyz>
+        <xyz>0.0 -1 0.0</xyz>
+        <limit>
+            <lower>0</lower>
+            <upper>2.460914245</upper>
+        </limit>
       </axis>
     </joint>
@@ -580,5 +660,16 @@
       <axis>
         <xyz>0.0 1 0.0</xyz>
-      </axis>
+        <limit>
+            <lower>-1.651081472</lower>
+            <upper>1.780235837</upper>
+        </limit>
+      </axis>
+      <axis2>
+        <xyz>0.0 0.0 1.0</xyz>
+        <limit>
+            <lower>-0.438077642</lower>
+            <upper>0.808087444</upper>
+        </limit>
+      </axis2>
     </joint>
     <link name='${prefix}right_hand'>
@@ -619,5 +710,16 @@
       <axis>
         <xyz>0.0 1 0.0</xyz>
-      </axis>
+        <limit>
+            <lower>-1.651081472</lower>
+            <upper>1.780235837</upper>
+        </limit>
+      </axis>
+      <axis2>
+        <xyz>0.0 0.0 1.0</xyz>
+        <limit>
+            <lower>-0.438077642</lower>
+            <upper>0.808087444</upper>
+        </limit>
+      </axis2>
     </joint>
 </xacro:macro>

Commit message: Add damping. Fix shoulder joints

File: human-model-include.xacro (robot description, xacro)
@@ -86,4 +86,7 @@
           <upper>0.726056969</upper>
         </limit>
+        <dynamics>
+            <damping>0.2</damping>
+        </dynamics>
       </axis>
     </joint>
@@ -142,4 +145,7 @@
           <upper>0.726056969</upper>
         </limit>
+        <dynamics>
+            <damping>0.2</damping>
+        </dynamics>
       </axis>
     </joint>
@@ -185,4 +191,7 @@
           <upper>2.160717614</upper>
         </limit>
+        <dynamics>
+            <damping>0.2</damping>
+        </dynamics>
       </axis>
     </joint>
@@ -228,4 +237,7 @@
           <upper>2.160717614</upper>
         </limit>
+        <dynamics>
+            <damping>0.2</damping>
+        </dynamics>
       </axis>
     </joint>
@@ -271,4 +283,7 @@
             <upper>0</upper>
         </limit>
+        <dynamics>
+            <damping>0.2</damping>
+        </dynamics>
       </axis>
       <axis2>
@@ -278,4 +293,7 @@
             <upper>1.012290966</upper>
         </limit>
+        <dynamics>
+            <damping>0.2</damping>
+        </dynamics>
       </axis2>
     </joint>
@@ -321,4 +339,7 @@
             <upper>0</upper>
         </limit>
+        <dynamics>
+            <damping>0.2</damping>
+        </dynamics>
       </axis>
       <axis2>
@@ -328,4 +349,7 @@
             <upper>1.012290966</upper>
         </limit>
+        <dynamics>
+            <damping>0.2</damping>
+        </dynamics>
       </axis2>
     </joint>
@@ -360,4 +384,7 @@
             <upper>0</upper>
         </limit>
+        <dynamics>
+            <damping>0.0</damping>
+        </dynamics>
       </axis>
     </joint>
@@ -372,4 +399,7 @@
             <upper>0</upper>
         </limit>
+        <dynamics>
+            <damping>0.0</damping>
+        </dynamics>
       </axis>
     </joint>
@@ -404,4 +434,7 @@
             <upper>0</upper>
         </limit>
+        <dynamics>
+            <damping>0.0</damping>
+        </dynamics>
       </axis>
     </joint>
@@ -473,16 +506,22 @@
       <pose>0.0 0.0 -0.151 0.0 0.0 0.0</pose>
       <axis>
-        <xyz>0.0 1 0.0</xyz>
+        <xyz>0.0 1.0 0.0</xyz>
         <limit>
             <lower>-3.371976115</lower>
             <upper>1.099557429</upper>
         </limit>
+        <dynamics>
+            <damping>0.2</damping>
+        </dynamics>
       </axis>
       <axis2>
-        <xyz>0.0 0.0 -1.0</xyz>
+        <xyz>-1.0 0.0 0.0</xyz>
         <limit>
             <lower>-2.305579942</lower>
             <upper>0.88662726</upper>
         </limit>
+        <dynamics>
+            <damping>0.2</damping>
+        </dynamics>
       </axis2>
     </joint>
@@ -523,16 +562,22 @@
       <pose>0.0 0.0 -0.151 0.0 0.0 0.0</pose>
       <axis>
-        <xyz>0.0 1 0.0</xyz>
+        <xyz>0.0 1.0 0.0</xyz>
         <limit>
             <lower>-3.371976115</lower>
             <upper>1.099557429</upper>
         </limit>
+        <dynamics>
+            <damping>0.2</damping>
+        </dynamics>
       </axis>
       <axis2>
-        <xyz>0.0 0.0 1.0</xyz>
+        <xyz>1.0 0.0 0.0</xyz>
         <limit>
             <lower>-2.305579942</lower>
             <upper>0.88662726</upper>
         </limit>
+        <dynamics>
+            <damping>0.2</damping>
+        </dynamics>
       </axis2>
     </joint>
@@ -578,4 +623,7 @@
             <upper>2.460914245</upper>
         </limit>
+        <dynamics>
+            <damping>0.2</damping>
+        </dynamics>
       </axis>
     </joint>
@@ -621,4 +669,7 @@
             <upper>2.460914245</upper>
         </limit>
+        <dynamics>
+            <damping>0.2</damping>
+        </dynamics>
       </axis>
     </joint>
@@ -664,4 +715,7 @@
             <upper>1.780235837</upper>
         </limit>
+        <dynamics>
+            <damping>0.2</damping>
+        </dynamics>
       </axis>
       <axis2>
@@ -671,4 +725,7 @@
             <upper>0.808087444</upper>
         </limit>
+        <dynamics>
+            <damping>0.2</damping>
+        </dynamics>
       </axis2>
     </joint>
@@ -714,4 +771,7 @@
             <upper>1.780235837</upper>
         </limit>
+        <dynamics>
+            <damping>0.2</damping>
+        </dynamics>
       </axis>
       <axis2>
@@ -721,4 +781,7 @@
             <upper>0.808087444</upper>
         </limit>
+        <dynamics>
+            <damping>0.2</damping>
+        </dynamics>
       </axis2>
     </joint>
