Commit message: Add contact sensors to all links

File: human-model-include.xacro (robot description, xacro)
@@ -31,4 +31,9 @@
         </geometry>
        </visual>
+       <sensor name='trunk_contact' type='contact'>
+          <contact>
+            <collision>collision</collision>
+          </contact>
+        </sensor>
     </link>
     <link name='${prefix}left_foot'>
@@ -180,4 +185,9 @@
         </geometry>
        </visual>
+       <sensor name='left_leg_contact' type='contact'>
+          <contact>
+            <collision>collision</collision>
+          </contact>
+        </sensor>
     </link>
     <joint name='${prefix}left_knee' type='revolute'>
@@ -226,4 +236,9 @@
         </geometry>
        </visual>
+       <sensor name='right_leg_contact' type='contact'>
+          <contact>
+            <collision>collision</collision>
+          </contact>
+        </sensor>
     </link>
     <joint name='${prefix}right_knee' type='revolute'>
@@ -272,4 +287,9 @@
         </geometry>
        </visual>
+       <sensor name='left_thigh_contact' type='contact'>
+          <contact>
+            <collision>collision</collision>
+          </contact>
+        </sensor>
     </link>
     <joint name='${prefix}left_hip' type='revolute'>
@@ -328,4 +348,9 @@
         </geometry>
        </visual>
+       <sensor name='right_thigh_contact' type='contact'>
+          <contact>
+            <collision>collision</collision>
+          </contact>
+        </sensor>
     </link>
     <joint name='${prefix}right_hip' type='revolute'>
@@ -373,4 +398,9 @@
         </geometry>
        </visual>
+       <sensor name='transpelvic_contact' type='contact'>
+          <contact>
+            <collision>collision</collision>
+          </contact>
+        </sensor>
     </link>
     <joint name='${prefix}lower_spine' type='revolute'>
@@ -423,4 +453,9 @@
         </geometry>
        </visual>
+       <sensor name='clavicular_link_contact' type='contact'>
+          <contact>
+            <collision>collision</collision>
+          </contact>
+        </sensor>
     </link>
     <joint name='${prefix}neck' type='revolute'>
@@ -469,4 +504,9 @@
         </geometry>
        </visual>
+       <sensor name='head_neck_contact' type='contact'>
+          <contact>
+            <collision>collision</collision>
+          </contact>
+        </sensor>
     </link>
     <link name='${prefix}left_upper_arm'>
@@ -500,4 +540,9 @@
         </geometry>
        </visual>
+       <sensor name='left_upper_arm_contact' type='contact'>
+          <contact>
+            <collision>collision</collision>
+          </contact>
+        </sensor>
     </link>
     <joint name='${prefix}left_shoulder' type='revolute'>
@@ -556,4 +601,9 @@
         </geometry>
        </visual>
+       <sensor name='right_upper_arm_contact' type='contact'>
+          <contact>
+            <collision>collision</collision>
+          </contact>
+        </sensor>
     </link>
     <joint name='${prefix}right_shoulder' type='revolute'>
@@ -612,4 +662,9 @@
         </geometry>
        </visual>
+       <sensor name='left_forearm_contact' type='contact'>
+          <contact>
+            <collision>collision</collision>
+          </contact>
+        </sensor>
     </link>
     <joint name='${prefix}left_elbow' type='revolute'>
@@ -658,4 +713,9 @@
         </geometry>
        </visual>
+       <sensor name='right_forearm_contact' type='contact'>
+          <contact>
+            <collision>collision</collision>
+          </contact>
+        </sensor>
     </link>
     <joint name='${prefix}right_elbow' type='revolute'>
@@ -704,4 +764,9 @@
         </geometry>
        </visual>
+       <sensor name='left_hand_contact' type='contact'>
+          <contact>
+            <collision>collision</collision>
+          </contact>
+        </sensor>
     </link>
     <joint name='${prefix}left_wrist' type='revolute'>
@@ -760,4 +825,9 @@
         </geometry>
        </visual>
+       <sensor name='right_hand_contact' type='contact'>
+          <contact>
+            <collision>collision</collision>
+          </contact>
+        </sensor>
     </link>
     <joint name='${prefix}right_wrist' type='revolute'>

Commit message: Add an initial velocity plugin. Fix the 2nd axies for joints. Fix the main axis for the hips

File: human-model-include.xacro (robot description, xacro)
@@ -293,5 +293,5 @@
         </sensor>
     </link>
-    <joint name='${prefix}left_hip' type='revolute'>
+    <joint name='${prefix}left_hip' type='revolute2'>
       <parent>${prefix}transpelvic_link</parent>
       <child>${prefix}left_thigh</child>
@@ -300,6 +300,6 @@
         <xyz>0.0 1 0.0</xyz>
         <limit>
-            <lower>-2.043780554</lower>
-            <upper>0</upper>
+            <lower>0</lower>
+            <upper>2.043780554</upper>
         </limit>
         <dynamics>
@@ -354,5 +354,5 @@
         </sensor>
     </link>
-    <joint name='${prefix}right_hip' type='revolute'>
+    <joint name='${prefix}right_hip' type='revolute2'>
       <parent>${prefix}transpelvic_link</parent>
       <child>${prefix}right_thigh</child>
@@ -361,6 +361,6 @@
         <xyz>0.0 1 0.0</xyz>
         <limit>
-            <lower>-2.043780554</lower>
-            <upper>0</upper>
+            <lower>0.0</lower>
+            <upper>2.043780554</upper>
         </limit>
         <dynamics>
@@ -546,5 +546,5 @@
         </sensor>
     </link>
-    <joint name='${prefix}left_shoulder' type='revolute'>
+    <joint name='${prefix}left_shoulder' type='revolute2'>
       <parent>${prefix}clavicular_link</parent>
       <child>${prefix}left_upper_arm</child>
@@ -607,5 +607,5 @@
         </sensor>
     </link>
-    <joint name='${prefix}right_shoulder' type='revolute'>
+    <joint name='${prefix}right_shoulder' type='revolute2'>
       <parent>${prefix}clavicular_link</parent>
       <child>${prefix}right_upper_arm</child>
@@ -770,5 +770,5 @@
         </sensor>
     </link>
-    <joint name='${prefix}left_wrist' type='revolute'>
+    <joint name='${prefix}left_wrist' type='revolute2'>
       <parent>${prefix}left_forearm</parent>
       <child>${prefix}left_hand</child>
@@ -831,5 +831,5 @@
         </sensor>
     </link>
-    <joint name='${prefix}right_wrist' type='revolute'>
+    <joint name='${prefix}right_wrist' type='revolute2'>
       <parent>${prefix}right_forearm</parent>
       <child>${prefix}right_hand</child>

File: human-model.xacro (robot description, xacro)
@@ -3,5 +3,5 @@
   <model name="human" xmlns:xacro="http://www.ros.org/wiki/xacro">
     <!-- TODO: These should not be needed but parameters aren't working -->
-    <!-- <xacro:property name="xoffset" value="0" /> -->
+    <xacro:property name="xoffset" value="0" />
     <xacro:property name="yoffset" value="0" />
     <xacro:property name="zoffset" value="0" />

Commit message: Fix left/right labeling issue

File: human-model-include.xacro (robot description, xacro)
@@ -37,5 +37,5 @@
         </sensor>
     </link>
-    <link name='${prefix}left_foot'>
+    <link name='${prefix}right_foot'>
       <pose>${0.041 + xoffset} ${-0.0855 + yoffset} ${0.0 + zoffset} 0.0 1.570796327 0.0</pose><!-- Move forward by half length of foot. Y coordinate is half the pelvic width. Rotate to horizontal plane -->
       <inertial>
@@ -75,13 +75,13 @@
         </geometry>
        </visual>
-       <sensor name='left_foot_contact' type='contact'>
-          <contact>
-            <collision>collision</collision>
-          </contact>
-        </sensor>
-    </link>
-    <joint name='${prefix}left_ankle' type='revolute'>
-      <parent>${prefix}left_leg</parent>
-      <child>${prefix}left_foot</child>
+       <sensor name='right_foot_contact' type='contact'>
+          <contact>
+            <collision>collision</collision>
+          </contact>
+        </sensor>
+    </link>
+    <joint name='${prefix}right_ankle' type='revolute'>
+      <parent>${prefix}right_leg</parent>
+      <child>${prefix}right_foot</child>
       <pose>0.0 0.0 0.0 0.0 1.570796327 0.0</pose>
       <axis>
@@ -96,5 +96,5 @@
       </axis>
     </joint>
-    <link name='${prefix}right_foot'>
+    <link name='${prefix}left_foot'>
       <pose>${0.041 + xoffset} ${0.0855 + yoffset} ${0.0 + zoffset} 0.0 1.570796327 0.0</pose><!-- Move forward by half length of foot. Y coordinate is half the pelvic width. Rotate to horizontal plane -->
       <inertial>
@@ -134,13 +134,13 @@
         </geometry>
        </visual>
-       <sensor name='right_foot_contact' type='contact'>
-          <contact>
-            <collision>collision</collision>
-          </contact>
-        </sensor>
-    </link>
-    <joint name='${prefix}right_ankle' type='revolute'>
-      <parent>${prefix}right_leg</parent>
-      <child>${prefix}right_foot</child>
+       <sensor name='left_foot_contact' type='contact'>
+          <contact>
+            <collision>collision</collision>
+          </contact>
+        </sensor>
+    </link>
+    <joint name='${prefix}left_ankle' type='revolute'>
+      <parent>${prefix}left_leg</parent>
+      <child>${prefix}left_foot</child>
       <pose>0.0 0.0 0.0 0.0 1.570796327 0.0</pose>
        <axis>
@@ -155,6 +155,57 @@
       </axis>
     </joint>
+    <link name='${prefix}right_leg'>
+      <pose>${0.0 + xoffset} ${-0.0855 + yoffset} ${0.2045 + zoffset} 0.0 0.0 0.0</pose><!-- Y coordinate is half the pelvic width. Z coordinate is half the leg height. -->
+      <inertial>
+        <mass>3.4689</mass>
+        <pose>0.0 0.0 0.027403 0.0 0.0 0.0</pose>
+        <inertia>
+          <ixx>0.052923954</ixx>
+          <iyy>0.000276446</iyy>
+          <izz>0.052923954</izz>
+          <ixy>0.0</ixy>
+          <ixz>0.0</ixz>
+          <iyz>0.0</iyz>
+        </inertia>
+      </inertial>
+      <collision name='collision'>
+        <geometry>
+          <cylinder>
+            <length>0.409</length>
+            <radius>0.02</radius>
+          </cylinder>
+        </geometry>
+       </collision>
+       <visual name='visual'>
+         <geometry>
+          <cylinder>
+            <length>0.409</length>
+            <radius>0.02</radius>
+          </cylinder>
+        </geometry>
+       </visual>
+       <sensor name='right_leg_contact' type='contact'>
+          <contact>
+            <collision>collision</collision>
+          </contact>
+        </sensor>
+    </link>
+    <joint name='${prefix}right_knee' type='revolute'>
+      <parent>${prefix}right_thigh</parent>
+      <child>${prefix}right_leg</child>
+      <pose>0.0 0.0 0.2045 0.0 0.0 0.0</pose>
+      <axis>
+        <xyz>0.0 1 0.0</xyz>
+        <limit>
+          <lower>0</lower>
+          <upper>2.160717614</upper>
+        </limit>
+        <dynamics>
+            <damping>0.20</damping>
+        </dynamics>
+      </axis>
+    </joint>
     <link name='${prefix}left_leg'>
-      <pose>${0.0 + xoffset} ${-0.0855 + yoffset} ${0.2045 + zoffset} 0.0 0.0 0.0</pose><!-- Y coordinate is half the pelvic width. Z coordinate is half the leg height. -->
+      <pose>${0.0 + xoffset} ${0.0855 + yoffset} ${0.2045 + zoffset} 0.0 0.0 0.0</pose><!-- Y coordinate is half the pelvic width. Z coordinate is half the leg height -->
       <inertial>
         <mass>3.4689</mass>
@@ -206,56 +257,5 @@
       </axis>
     </joint>
-    <link name='${prefix}right_leg'>
-      <pose>${0.0 + xoffset} ${0.0855 + yoffset} ${0.2045 + zoffset} 0.0 0.0 0.0</pose><!-- Y coordinate is half the pelvic width. Z coordinate is half the leg height -->
-      <inertial>
-        <mass>3.4689</mass>
-        <pose>0.0 0.0 0.027403 0.0 0.0 0.0</pose>
-        <inertia>
-          <ixx>0.052923954</ixx>
-          <iyy>0.000276446</iyy>
-          <izz>0.052923954</izz>
-          <ixy>0.0</ixy>
-          <ixz>0.0</ixz>
-          <iyz>0.0</iyz>
-        </inertia>
-      </inertial>
-      <collision name='collision'>
-        <geometry>
-          <cylinder>
-            <length>0.409</length>
-            <radius>0.02</radius>
-          </cylinder>
-        </geometry>
-       </collision>
-       <visual name='visual'>
-         <geometry>
-          <cylinder>
-            <length>0.409</length>
-            <radius>0.02</radius>
-          </cylinder>
-        </geometry>
-       </visual>
-       <sensor name='right_leg_contact' type='contact'>
-          <contact>
-            <collision>collision</collision>
-          </contact>
-        </sensor>
-    </link>
-    <joint name='${prefix}right_knee' type='revolute'>
-      <parent>${prefix}right_thigh</parent>
-      <child>${prefix}right_leg</child>
-      <pose>0.0 0.0 0.2045 0.0 0.0 0.0</pose>
-      <axis>
-        <xyz>0.0 1 0.0</xyz>
-        <limit>
-          <lower>0</lower>
-          <upper>2.160717614</upper>
-        </limit>
-        <dynamics>
-            <damping>0.20</damping>
-        </dynamics>
-      </axis>
-    </joint>
-    <link name='${prefix}left_thigh'>
+    <link name='${prefix}right_thigh'>
       <pose>${0.0 + xoffset} ${-0.0855 + yoffset} ${0.626 + zoffset} 0.0 0.0 0.0</pose><!-- Y coordinate is half the pelvic width. X coordinate is the leg height + 0.5 * thigh height -->
       <inertial>
@@ -287,4 +287,65 @@
         </geometry>
        </visual>
+       <sensor name='right_thigh_contact' type='contact'>
+          <contact>
+            <collision>collision</collision>
+          </contact>
+        </sensor>
+    </link>
+    <joint name='${prefix}right_hip' type='revolute2'>
+      <parent>${prefix}transpelvic_link</parent>
+      <child>${prefix}right_thigh</child>
+      <pose>0.0 0.0 0.217 0.0 0.0 0.0</pose> <!--Height leg + thigh -->
+      <axis>
+        <xyz>0.0 1 0.0</xyz>
+        <limit>
+            <lower>0</lower>
+            <upper>2.043780554</upper>
+        </limit>
+        <dynamics>
+            <damping>0.20</damping>
+        </dynamics>
+      </axis>
+     <axis2>
+        <xyz>1.0 0.0 0.0</xyz>
+        <limit>
+            <lower>-0.483456203</lower>
+            <upper>1.012290966</upper>
+        </limit>
+        <dynamics>
+            <damping>0.20</damping>
+        </dynamics>
+      </axis2>
+    </joint>
+    <link name='${prefix}left_thigh'>
+      <pose>${0.0 + xoffset} ${0.0855 + yoffset} ${0.626 + zoffset} 0.0 0.0 0.0</pose><!-- Y coordinate is half the pelvic width. X coordinate is the leg height + 0.5 * thigh height -->
+      <inertial>
+        <mass>7.46</mass>
+        <pose>0.0 0.0 0.029078 0.0 0.0 0.0</pose>
+        <inertia>
+          <ixx>0.146596409</ixx>
+          <iyy>0.001321394</iyy>
+          <izz>0.146596409</izz>
+          <ixy>0.0</ixy>
+          <ixz>0.0</ixz>
+          <iyz>0.0</iyz>
+        </inertia>
+      </inertial>
+      <collision name='collision'>
+        <geometry>
+          <cylinder>
+            <length>0.434</length>
+            <radius>0.02</radius>
+          </cylinder>
+        </geometry>
+       </collision>
+       <visual name='visual'>
+         <geometry>
+          <cylinder>
+            <length>0.434</length>
+            <radius>0.02</radius>
+          </cylinder>
+        </geometry>
+       </visual>
        <sensor name='left_thigh_contact' type='contact'>
           <contact>
@@ -296,65 +357,4 @@
       <parent>${prefix}transpelvic_link</parent>
       <child>${prefix}left_thigh</child>
-      <pose>0.0 0.0 0.217 0.0 0.0 0.0</pose> <!--Height leg + thigh -->
-      <axis>
-        <xyz>0.0 1 0.0</xyz>
-        <limit>
-            <lower>0</lower>
-            <upper>2.043780554</upper>
-        </limit>
-        <dynamics>
-            <damping>0.20</damping>
-        </dynamics>
-      </axis>
-     <axis2>
-        <xyz>1.0 0.0 0.0</xyz>
-        <limit>
-            <lower>-0.483456203</lower>
-            <upper>1.012290966</upper>
-        </limit>
-        <dynamics>
-            <damping>0.20</damping>
-        </dynamics>
-      </axis2>
-    </joint>
-    <link name='${prefix}right_thigh'>
-      <pose>${0.0 + xoffset} ${0.0855 + yoffset} ${0.626 + zoffset} 0.0 0.0 0.0</pose><!-- Y coordinate is half the pelvic width. X coordinate is the leg height + 0.5 * thigh height -->
-      <inertial>
-        <mass>7.46</mass>
-        <pose>0.0 0.0 0.029078 0.0 0.0 0.0</pose>
-        <inertia>
-          <ixx>0.146596409</ixx>
-          <iyy>0.001321394</iyy>
-          <izz>0.146596409</izz>
-          <ixy>0.0</ixy>
-          <ixz>0.0</ixz>
-          <iyz>0.0</iyz>
-        </inertia>
-      </inertial>
-      <collision name='collision'>
-        <geometry>
-          <cylinder>
-            <length>0.434</length>
-            <radius>0.02</radius>
-          </cylinder>
-        </geometry>
-       </collision>
-       <visual name='visual'>
-         <geometry>
-          <cylinder>
-            <length>0.434</length>
-            <radius>0.02</radius>
-          </cylinder>
-        </geometry>
-       </visual>
-       <sensor name='right_thigh_contact' type='contact'>
-          <contact>
-            <collision>collision</collision>
-          </contact>
-        </sensor>
-    </link>
-    <joint name='${prefix}right_hip' type='revolute2'>
-      <parent>${prefix}transpelvic_link</parent>
-      <child>${prefix}right_thigh</child>
       <pose>0.0 0.0 0.217 0.0 0.0 0.0</pose> <!-- leg + thigh height -->
       <axis>
@@ -510,6 +510,67 @@
         </sensor>
     </link>
+    <link name='${prefix}right_upper_arm'>
+      <pose>${0.0 + xoffset} ${-0.0815 + yoffset} ${1.37 + zoffset} 0.0 0.0 0.0</pose><!-- Y coordinate is half the pelvic width. Z coordinate is leg + thigh + trunk + 0.5 * upper arm -->
+      <inertial>
+        <mass>2.0888</mass>
+        <pose>0.0 0.0 -0.019328 0.0 0.0 0.0</pose>
+        <inertia>
+          <ixx>0.019752519</ixx>
+          <iyy>9.28219E-05</iyy>
+          <izz>0.019752519</izz>
+          <ixy>0.0</ixy>
+          <ixz>0.0</ixz>
+          <iyz>0.0</iyz>
+        </inertia>
+      </inertial>
+      <collision name='collision'>
+        <geometry>
+          <cylinder>
+            <length>0.302</length>
+            <radius>0.02</radius>
+          </cylinder>
+        </geometry>
+       </collision>
+       <visual name='visual'>
+         <geometry>
+          <cylinder>
+            <length>0.302</length>
+            <radius>0.02</radius>
+          </cylinder>
+        </geometry>
+       </visual>
+       <sensor name='right_upper_arm_contact' type='contact'>
+          <contact>
+            <collision>collision</collision>
+          </contact>
+        </sensor>
+    </link>
+    <joint name='${prefix}right_shoulder' type='revolute2'>
+      <parent>${prefix}clavicular_link</parent>
+      <child>${prefix}right_upper_arm</child>
+      <pose>0.0 0.0 -0.151 0.0 0.0 0.0</pose>
+      <axis>
+        <xyz>0.0 1.0 0.0</xyz>
+        <limit>
+            <lower>-3.371976115</lower>
+            <upper>1.099557429</upper>
+        </limit>
+        <dynamics>
+            <damping>0.20</damping>
+        </dynamics>
+      </axis>
+      <axis2>
+        <xyz>1.0 0.0 0.0</xyz>
+        <limit>
+            <lower>-2.305579942</lower>
+            <upper>0.88662726</upper>
+        </limit>
+        <dynamics>
+            <damping>0.20</damping>
+        </dynamics>
+      </axis2>
+    </joint>
     <link name='${prefix}left_upper_arm'>
-      <pose>${0.0 + xoffset} ${-0.0815 + yoffset} ${1.37 + zoffset} 0.0 0.0 0.0</pose><!-- Y coordinate is half the pelvic width. Z coordinate is leg + thigh + trunk + 0.5 * upper arm -->
+      <pose>${0.0 + xoffset} ${0.0815 + yoffset} ${1.37 + zoffset} 0.0 0.0 0.0</pose><!-- Y coordinate is half the pelvic width. Z coordinate is leg + thigh + trunk + 0.5 * upper arm -->
       <inertial>
         <mass>2.0888</mass>
@@ -571,67 +632,57 @@
       </axis2>
     </joint>
-    <link name='${prefix}right_upper_arm'>
-      <pose>${0.0 + xoffset} ${0.0815 + yoffset} ${1.37 + zoffset} 0.0 0.0 0.0</pose><!-- Y coordinate is half the pelvic width. Z coordinate is leg + thigh + trunk + 0.5 * upper arm -->
-      <inertial>
-        <mass>2.0888</mass>
-        <pose>0.0 0.0 -0.019328 0.0 0.0 0.0</pose>
-        <inertia>
-          <ixx>0.019752519</ixx>
-          <iyy>9.28219E-05</iyy>
-          <izz>0.019752519</izz>
-          <ixy>0.0</ixy>
-          <ixz>0.0</ixz>
-          <iyz>0.0</iyz>
-        </inertia>
-      </inertial>
-      <collision name='collision'>
-        <geometry>
-          <cylinder>
-            <length>0.302</length>
-            <radius>0.02</radius>
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