Commit message: Reduce friction so model is more solvable with PR2 constraint. Fix shoulder joint limits

File: human-model-include.xacro (robot description, xacro)
@@ -61,6 +61,6 @@
           <friction>
             <ode>
-              <mu>100.0</mu>
-              <mu2>100.0</mu2>
+              <mu>1.0</mu>
+              <mu2>1.0</mu2>
             </ode>
           </friction>
@@ -120,6 +120,6 @@
           <friction>
             <ode>
-              <mu>100.0</mu>
-              <mu2>100.0</mu2>
+              <mu>1.0</mu>
+              <mu2>1.0</mu2>
             </ode>
           </friction>
@@ -298,5 +298,5 @@
       <pose>0.0 0.0 0.217 0.0 0.0 0.0</pose> <!--Height leg + thigh -->
       <axis>
-        <xyz>0.0 1 0.0</xyz>
+        <xyz>0.0 1.0 0.0</xyz>
         <limit>
             <lower>0</lower>
@@ -317,4 +317,17 @@
         </dynamics>
       </axis2>
+      <!-- Joint limits on ball joints not currently supported in gazebo -->
+      <!--
+      <axis3>
+        <xyz>0.0 0.0 1.0</xyz>
+        <limit>
+            <lower>-0.60562925</lower>
+            <upper>0.675442421</upper>
+        </limit>
+        <dynamics>
+            <damping>0.20</damping>
+        </dynamics>
+      </axis3>
+      -->
     </joint>
     <link name='${prefix}left_thigh'>
@@ -378,4 +391,17 @@
         </dynamics>
       </axis2>
+      <!-- Joint limits on ball joints not currently supported in gazebo -->
+      <!--
+     <axis3>
+        <xyz>0.0 0.0 -1.0</xyz>
+        <limit>
+            <lower>-0.60562925</lower>
+            <upper>0.675442421</upper>
+        </limit>
+        <dynamics>
+            <damping>0.20</damping>
+        </dynamics>
+      </axis3>
+      -->
     </joint>
     <link name='${prefix}transpelvic_link'>
@@ -553,6 +579,6 @@
         <xyz>0.0 1.0 0.0</xyz>
         <limit>
-            <lower>-3.371976115</lower>
-            <upper>1.099557429</upper>
+            <lower>-1.099557429</lower>
+            <upper>3.371976115</upper>
         </limit>
         <dynamics>
@@ -570,4 +596,17 @@
         </dynamics>
       </axis2>
+      <!-- Joint limits on ball joints not currently supported in gazebo -->
+      <!--
+     <axis3>
+        <xyz>0.0 0.0 1.0</xyz>
+        <limit>
+            <lower>-2.305579942</lower>
+            <upper>0.88662726</upper>
+        </limit>
+        <dynamics>
+            <damping>0.20</damping>
+        </dynamics>
+      </axis3>
+      -->
     </joint>
     <link name='${prefix}left_upper_arm'>
@@ -614,6 +653,6 @@
         <xyz>0.0 1.0 0.0</xyz>
         <limit>
-            <lower>-3.371976115</lower>
-            <upper>1.099557429</upper>
+            <lower>-1.099557429</lower>
+            <upper>3.371976115</upper>
         </limit>
         <dynamics>
@@ -631,4 +670,17 @@
         </dynamics>
       </axis2>
+      <!-- Joint limits on ball joints not currently supported in gazebo -->
+      <!--
+     <axis3>
+        <xyz>0.0 0.0 -1.0</xyz>
+        <limit>
+            <lower>-2.305579942</lower>
+            <upper>0.88662726</upper>
+        </limit>
+        <dynamics>
+            <damping>0.20</damping>
+        </dynamics>
+      </axis3>
+      -->
     </joint>
     <link name='${prefix}right_forearm'>
