Commit message: Get stable controlled plugin working for all right arm joints

File: pr2-include.xacro (robot description, xacro)
@@ -97,10 +97,4 @@
           <topic>__default_topic__</topic>
         </contact>
-        <plugin name='base_gazebo_ros_bumper_controller' filename='libgazebo_ros_bumper.so'>
-          <alwaysOn>true</alwaysOn>
-          <updateRate>100.0</updateRate>
-          <bumperTopicName>base_bumper</bumperTopicName>
-          <frameName>world</frameName>
-        </plugin>
         <pose>0 0 0.051 0 -0 0</pose>
       </sensor>
@@ -1024,10 +1018,4 @@
         </contact>
         <update_rate>100</update_rate>
-        <plugin name='torso_lift_gazebo_ros_bumper_controller' filename='libgazebo_ros_bumper.so'>
-          <alwaysOn>true</alwaysOn>
-          <updateRate>100.0</updateRate>
-          <bumperTopicName>torso_lift_bumper</bumperTopicName>
-          <frameName>world</frameName>
-        </plugin>
       </sensor>
     </link>
@@ -2076,10 +2064,4 @@
           <topic>__default_topic__</topic>
         </contact>
-        <plugin name='l_gripper_l_finger_tip_gazebo_ros_bumper_controller' filename='libgazebo_ros_bumper.so'>
-          <alwaysOn>true</alwaysOn>
-          <frameName>l_gripper_l_finger_tip_link</frameName>
-          <updateRate>100.0</updateRate>
-          <bumperTopicName>l_gripper_l_finger_tip_bumper</bumperTopicName>
-        </plugin>
       </sensor>
     </link>
@@ -2332,10 +2314,4 @@
           <topic>__default_topic__</topic>
         </contact>
-        <plugin name='l_gripper_r_finger_tip_gazebo_ros_bumper_controller' filename='libgazebo_ros_bumper.so'>
-          <alwaysOn>true</alwaysOn>
-          <frameName>l_gripper_r_finger_tip_link</frameName>
-          <updateRate>100.0</updateRate>
-          <bumperTopicName>l_gripper_r_finger_tip_bumper</bumperTopicName>
-        </plugin>
       </sensor>
     </link>
@@ -3250,10 +3226,4 @@
           <topic>__default_topic__</topic>
         </contact>
-        <plugin name='r_gripper_l_finger_tip_gazebo_ros_bumper_controller' filename='libgazebo_ros_bumper.so'>
-          <alwaysOn>true</alwaysOn>
-          <frameName>r_gripper_l_finger_tip_link</frameName>
-          <updateRate>100.0</updateRate>
-          <bumperTopicName>r_gripper_l_finger_tip_bumper</bumperTopicName>
-        </plugin>
       </sensor>
     </link>
@@ -3506,10 +3476,4 @@
           <topic>__default_topic__</topic>
         </contact>
-        <plugin name='r_gripper_r_finger_tip_gazebo_ros_bumper_controller' filename='libgazebo_ros_bumper.so'>
-          <alwaysOn>true</alwaysOn>
-          <frameName>r_gripper_r_finger_tip_link</frameName>
-          <updateRate>100.0</updateRate>
-          <bumperTopicName>r_gripper_r_finger_tip_bumper</bumperTopicName>
-        </plugin>
       </sensor>
     </link>
@@ -3580,32 +3544,4 @@
       </axis>
     </joint>
-    <plugin name='gazebo_ros_controller_manager' filename='libgazebo_ros_controller_manager.so'>
-      <alwaysOn>true</alwaysOn>
-      <updateRate>1000.0</updateRate>
-    </plugin>
-    <plugin name='gazebo_ros_power_monitor_controller' filename='libgazebo_ros_power_monitor.so'>
-      <alwaysOn>true</alwaysOn>
-      <updateRate>1.0</updateRate>
-      <timeout>5</timeout>
-      <powerStateTopic>power_state</powerStateTopic>
-      <powerStateRate>10.0</powerStateRate>
-      <fullChargeCapacity>87.78</fullChargeCapacity>
-      <dischargeRate>-474</dischargeRate>
-      <chargeRate>525</chargeRate>
-      <dischargeVoltage>15.52</dischargeVoltage>
-      <chargeVoltage>16.41</chargeVoltage>
-    </plugin>
-    <plugin name='p3d_base_controller' filename='libgazebo_ros_p3d.so'>
-      <alwaysOn>true</alwaysOn>
-      <updateRate>100.0</updateRate>
-      <topicName>base_pose_ground_truth</topicName>
-      <gaussianNoise>0.01</gaussianNoise>
-      <frameName>map</frameName>
-      <xyzOffsets>0 0 0</xyzOffsets>
-      <rpyOffsets>0 0 0</rpyOffsets>
-      <bodyName>base_footprint</bodyName>
-      <xyzOffset>0 0 -0.051</xyzOffset>
-      <rpyOffset>0 -0 0</rpyOffset>
-    </plugin>
     <joint name='torso_lift_screw_torso_lift_joint' type='screw'>
       <parent>torso_lift_link</parent>
@@ -3621,39 +3557,4 @@
       <thread_pitch>3141.6</thread_pitch>
     </joint>
-    <plugin name='imu_controller' filename='libgazebo_ros_imu.so'>
-      <alwaysOn>true</alwaysOn>
-      <updateRate>100.0</updateRate>
-      <topicName>torso_lift_imu/data</topicName>
-      <gaussianNoise>2.89e-08</gaussianNoise>
-      <serviceName>/default_imu</serviceName>
-      <bodyName>torso_lift_link</bodyName>
-      <xyzOffset>0.02977 0.1497 -0.164</xyzOffset>
-      <rpyOffset>0 -2.06701e-13 0</rpyOffset>
-    </plugin>
-    <plugin name='projector_wg6802418_controller' filename='libgazebo_ros_projector.so'>
-      <alwaysOn>true</alwaysOn>
-      <updateRate>15.0</updateRate>
-      <textureName>stereo_projection_pattern_high_res_red.png</textureName>
-      <filterTextureName>stereo_projection_pattern_filter.png</filterTextureName>
-      <textureTopicName>projector_wg6802418_controller/image</textureTopicName>
-      <projectorTopicName>projector_wg6802418_controller/projector</projectorTopicName>
-      <projector>head_tilt_link/projector_wg6802418_projector_wg6802418</projector>
-    </plugin>
-    <plugin name='p3d_r_gripper_l_finger_controller' filename='libgazebo_ros_p3d.so'>
-      <alwaysOn>true</alwaysOn>
-      <updateRate>100.0</updateRate>
-      <bodyName>r_gripper_l_finger_link</bodyName>
-      <topicName>r_gripper_l_finger_pose_ground_truth</topicName>
-      <gaussianNoise>0.0</gaussianNoise>
-      <frameName>base_footprint</frameName>
-      <xyzOffset>0 0 -0.051</xyzOffset>
-      <rpyOffset>0 -0 0</rpyOffset>
-    </plugin>
-    <plugin name='f3d_r_gripper_l_finger_controller' filename='libgazebo_ros_f3d.so'>
-      <alwaysOn>true</alwaysOn>
-      <updateRate>100.0</updateRate>
-      <bodyName>r_gripper_l_finger_link</bodyName>
-      <topicName>r_gripper_l_finger_force_ground_truth</topicName>
-    </plugin>
     <link name='r_gripper_l_parallel_link'>
       <inertial>
@@ -3796,16 +3697,4 @@
       </axis>
     </joint>
-    <plugin name='p3d_r_gripper_palm_controller' filename='libgazebo_ros_p3d.so'>
-      <alwaysOn>true</alwaysOn>
-      <updateRate>100.0</updateRate>
-      <topicName>r_gripper_palm_pose_ground_truth</topicName>
-      <xyzOffsets>0 0 0</xyzOffsets>
-      <rpyOffsets>0 0 0</rpyOffsets>
-      <gaussianNoise>0.0</gaussianNoise>
-      <frameName>map</frameName>
-      <bodyName>r_wrist_roll_link</bodyName>
-      <xyzOffset>0 0 0</xyzOffset>
-      <rpyOffset>0 -0 0</rpyOffset>
-    </plugin>
     <gripper name='r_grasp_hack'>
       <grasp_check>
@@ -3818,20 +3707,4 @@
       <palm_link>r_wrist_roll_link</palm_link>
     </gripper>
-    <plugin name='p3d_l_gripper_l_finger_controller' filename='libgazebo_ros_p3d.so'>
-      <alwaysOn>true</alwaysOn>
-      <updateRate>100.0</updateRate>
-      <bodyName>l_gripper_l_finger_link</bodyName>
-      <topicName>l_gripper_l_finger_pose_ground_truth</topicName>
-      <gaussianNoise>0.0</gaussianNoise>
-      <frameName>base_footprint</frameName>
-      <xyzOffset>0 0 -0.051</xyzOffset>
-      <rpyOffset>0 -0 0</rpyOffset>
-    </plugin>
-    <plugin name='f3d_l_gripper_l_finger_controller' filename='libgazebo_ros_f3d.so'>
-      <alwaysOn>true</alwaysOn>
-      <updateRate>100.0</updateRate>
-      <bodyName>l_gripper_l_finger_link</bodyName>
-      <topicName>l_gripper_l_finger_force_ground_truth</topicName>
-    </plugin>
     <link name='l_gripper_l_parallel_link'>
       <inertial>
@@ -3975,16 +3848,4 @@
     </joint>
     <static>0</static>
-    <plugin name='p3d_l_gripper_palm_controller' filename='libgazebo_ros_p3d.so'>
-      <alwaysOn>true</alwaysOn>
-      <updateRate>100.0</updateRate>
-      <topicName>l_gripper_palm_pose_ground_truth</topicName>
-      <xyzOffsets>0 0 0</xyzOffsets>
-      <rpyOffsets>0 0 0</rpyOffsets>
-      <gaussianNoise>0.0</gaussianNoise>
-      <frameName>map</frameName>
-      <bodyName>l_wrist_roll_link</bodyName>
-      <xyzOffset>0 0 0</xyzOffset>
-      <rpyOffset>0 -0 0</rpyOffset>
-    </plugin>
     <gripper name='l_grasp_hack'>
       <grasp_check>
@@ -3997,3 +3858,12 @@
       <palm_link>l_wrist_roll_link</palm_link>
     </gripper>
+    <plugin name="pr2_arm_controller" filename="libStableControllerPlugin.dylib">
+      <controlled-joint>r_shoulder_lift_joint</controlled-joint>
+      <controlled-joint>r_shoulder_pan_joint</controlled-joint>
+      <controlled-joint>r_upper_arm_roll_joint</controlled-joint>
+      <controlled-joint>r_elbow_flex_joint</controlled-joint>
+      <controlled-joint>r_forearm_roll_joint</controlled-joint>
+      <controlled-joint>r_wrist_flex_joint</controlled-joint>
+      <controlled-joint>r_wrist_roll_joint</controlled-joint>
+    </plugin>
 </sdf>

File: pr2.xacro (robot description, xacro)
@@ -1,5 +1,5 @@
 <sdf version="1.5">
   <model name="pr2" xmlns:xacro="http://www.ros.org/wiki/xacro">
-   <xacro:property name="armEffort" value="0" /> <!-- Standard value is 30 -->
+   <xacro:property name="armEffort" value="100" /> <!-- Standard value is 30 -->
     <xacro:property name="wristEffort" value="0" /> <!-- Standard value is 10 -->
     <xacro:include filename="pr2-include.xacro" />
