Commit message: Finish getting model files auto built

File: models/combined-human-pr2/combined-human-pr2.xacro (robot description, xacro)
@@ -3,5 +3,5 @@
    <xacro:property name="armEffort" value="0" /> <!-- Standard value is 30 -->
     <xacro:property name="wristEffort" value="0" /> <!-- Standard value is 10 -->
-    <xacro:include filename="pr2-include.xacro" />
+    <xacro:include filename="../pr2/pr2.include" />
     <!-- Controller for the pr2 arm -->
     <!-- <plugin name="pr2_arm_controller" filename="libStableControllerPlugin.dylib">    </plugin>-->
@@ -12,5 +12,5 @@
     <xacro:property name="zoffset" value="0" />
     <xacro:property name="prefix" value="" />
-    <xacro:include filename="human-model-include.xacro"/>
+    <xacro:include filename="../human/human.include"/>
     <!-- Virtual connecting joint -->
     <joint name="virtual_robot_human_connection" type="ball">

File: models/human/human.xacro (robot description, xacro)
@@ -8,5 +8,5 @@
     <xacro:property name="prefix" value="" />
     <static>false</static>
-    <xacro:include filename="human-model-include.xacro"/>
+    <xacro:include filename="human.include"/>
     <!-- <xacro:human xoffset="0" yoffset="0" zoffset="0.0"/>--> <!-- Base pose -->
   </model>

File: models/pr2/pr2.xacro (robot description, xacro)
@@ -1,7 +1,7 @@
 <sdf version="1.5">
   <model name="pr2" xmlns:xacro="http://www.ros.org/wiki/xacro">
-   <xacro:property name="armEffort" value="100" /> <!-- Standard value is 30 -->
+   <xacro:property name="armEffort" value="0" /> <!-- Standard value is 30 -->
     <xacro:property name="wristEffort" value="0" /> <!-- Standard value is 10 -->
-    <xacro:include filename="pr2-include.xacro" />
+    <xacro:include filename="pr2.include" />
     <!-- Controller for the pr2 arm -->
     <!-- <plugin name="pr2_arm_controller" filename="libStableControllerPlugin.dylib">    </plugin>-->
