Commit message: Rewrite the contact forces listener to be a plugin

File: models/pr2/pr2.xacro (robot description, xacro)
@@ -1,9 +1,7 @@
 <sdf version="1.5">
   <model name="pr2" xmlns:xacro="http://www.ros.org/wiki/xacro">
-   <xacro:property name="armEffort" value="0" /> <!-- Standard value is 30 -->
-    <xacro:property name="wristEffort" value="0" /> <!-- Standard value is 10 -->
+   <xacro:property name="armEffort" value="30" /> <!-- Standard value is 30 -->
+    <xacro:property name="wristEffort" value="10" /> <!-- Standard value is 10 -->
     <xacro:include filename="pr2.include" />
-    <!-- Controller for the pr2 arm -->
-    <!-- <plugin name="pr2_arm_controller" filename="libStableControllerPlugin.dylib">    </plugin>-->
   </model>
 </sdf>
