Commit message: Final work on framework

File: models/combined-human-pr2-zero-effort/combined-human-pr2.xacro (robot description, xacro)
@@ -1,6 +1,6 @@
 <sdf version="1.5">
   <model name="human" xmlns:xacro="http://www.ros.org/wiki/xacro">
-   <xacro:property name="armEffort" value="30" /> <!-- Standard value is 30 -->
-   <xacro:property name="wristEffort" value="10" /> <!-- Standard value is 10 -->
+   <xacro:property name="armEffort" value="0" /> <!-- Standard value is 30 -->
+   <xacro:property name="wristEffort" value="0" /> <!-- Standard value is 10 -->
    <xacro:include filename="../pr2/pr2.include" />
     <!-- TODO: Get these working -->

Commit message: Move biped closer to human

File: models/combined-human-pr2-zero-effort/combined-human-pr2.xacro (robot description, xacro)
@@ -4,14 +4,10 @@
    <xacro:property name="wristEffort" value="0" /> <!-- Standard value is 10 -->
    <xacro:include filename="../pr2/pr2.include" />
-    <!-- TODO: Get these working -->
-    <xacro:property name="xoffset" value="0.939280" />
-    <xacro:property name="yoffset" value="-0.25" />
+    <xacro:property name="xoffset" value="0.739280" />
+    <xacro:property name="yoffset" value="0" />
     <xacro:property name="zoffset" value="0" />
     <xacro:property name="prefix" value="" />
    <!-- Human -->
    <xacro:include filename="../human/human.include"/>
-   <!-- Virtual connecting joint -->
-   <!-- Joint is added dynamically -->
-   <!-- <xacro:include filename="../combined-human-pr2/connecting-joint.include" />-->
   </model>
 </sdf>

File: models/combined-human-pr2/combined-human-pr2.xacro (robot description, xacro)
@@ -5,13 +5,10 @@
    <xacro:include filename="../pr2/pr2.include" />
     <!-- TODO: Get these working -->
-    <xacro:property name="xoffset" value="0.939280" />
-    <xacro:property name="yoffset" value="-0.25" />
+    <xacro:property name="xoffset" value="0.739280" />
+    <xacro:property name="yoffset" value="0" />
     <xacro:property name="zoffset" value="0" />
     <xacro:property name="prefix" value="" />
    <!-- Human -->
    <xacro:include filename="../human/human.include"/>
-   <!-- Virtual connecting joint -->
-   <!-- Joint is added dynamically -->
-   <!-- <xacro:include filename="../combined-human-pr2/connecting-joint.include" />-->
   </model>
 </sdf>
