Commit message: Update design weight for calibration

File: models/arm-calibration/pr2-calibration.xacro (robot description, xacro)
@@ -9,5 +9,5 @@
        <pose>0.84791 -0.188 0.790675 0.0 0.0 0.0</pose>
        <inertial>
-          <mass>3</mass>
+          <mass>4.0</mass> <!-- Max design support weight of arm -->
           <pose>0.0 0.0 0.0 0.0 0.0 0.0</pose><!-- Link mass is centered -->
        </inertial>

Commit message: Add locked arms. Add feature to delay control of arms

File: models/arm-calibration/pr2-calibration.xacro (robot description, xacro)
@@ -3,4 +3,5 @@
    <xacro:property name="armEffort" value="30" /> <!-- Standard value is 30 -->
    <xacro:property name="wristEffort" value="10" /> <!-- Standard value is 10 -->
+   <xacro:property name="jointFriction" value="0" />
    <xacro:include filename="../pr2/pr2.include" />
    <!-- Add a weight to the pr2 arm -->

File: models/combined-human-pr2-zero-effort/combined-human-pr2.xacro (robot description, xacro)
@@ -3,4 +3,5 @@
    <xacro:property name="armEffort" value="0" /> <!-- Standard value is 30 -->
    <xacro:property name="wristEffort" value="0" /> <!-- Standard value is 10 -->
+   <xacro:property name="jointFriction" value="0" />
    <xacro:include filename="../pr2/pr2.include" />
     <xacro:property name="xoffset" value="0.739280" />

File: models/locked-arms/locked-arms.xacro (robot description, xacro)
@@ -1,7 +1,7 @@
 <sdf version="1.5">
   <model name="human" xmlns:xacro="http://www.ros.org/wiki/xacro">
-   <xacro:property name="armEffort" value="30" /> <!-- Standard value is 30 -->
-   <xacro:property name="wristEffort" value="10" /> <!-- Standard value is 10 -->
-   <xacro:property name="jointFriction" value="0" />
+   <xacro:property name="armEffort" value="0" /> <!-- Standard value is 30 -->
+   <xacro:property name="wristEffort" value="0" /> <!-- Standard value is 10 -->
+   <xacro:property name="jointFriction" value="500" />
    <xacro:include filename="../pr2/pr2.include" />
     <xacro:property name="xoffset" value="0.739280" />
@@ -12,5 +12,4 @@
    <xacro:include filename="../human/human.include"/>
    <plugin name="pr2_arm_controller" filename="libStableControllerPlugin.dylib">
-      <control-delay>0.0</control-delay>
       <controlled-joint>r_shoulder_lift_joint</controlled-joint>
       <controlled-joint>r_shoulder_pan_joint</controlled-joint>

File: models/pr2/pr2.xacro (robot description, xacro)
@@ -2,6 +2,7 @@
   <model name="pr2" xmlns:xacro="http://www.ros.org/wiki/xacro">
    <xacro:property name="armEffort" value="30" /> <!-- Standard value is 30 -->
-    <xacro:property name="wristEffort" value="10" /> <!-- Standard value is 10 -->
-    <xacro:include filename="pr2.include" />
+   <xacro:property name="wristEffort" value="10" /> <!-- Standard value is 10 -->
+   <xacro:property name="jointFriction" value="0" />
+   <xacro:include filename="pr2.include" />
   </model>
 </sdf>

Commit message: Recalibrate gains

File: models/arm-calibration/pr2-calibration.xacro (robot description, xacro)
@@ -10,5 +10,5 @@
        <pose>0.84791 -0.188 0.790675 0.0 0.0 0.0</pose>
        <inertial>
-          <mass>4.0</mass> <!-- Max design support weight of arm -->
+          <mass>1.8</mass> <!-- Max design support weight of arm -->
           <pose>0.0 0.0 0.0 0.0 0.0 0.0</pose><!-- Link mass is centered -->
        </inertial>
@@ -38,4 +38,21 @@
    <plugin name="calibration_plugin" filename="libArmCalibrationPlugin.dylib"/>
    <plugin name="joint_forces_plugin" filename="libJointForcesPlugin.dylib"/>
+   <plugin name="pr2_arm_controller" filename="libStableControllerPlugin.dylib">
+      <control-delay>0</control-delay>
+      <controlled-joint>r_shoulder_lift_joint</controlled-joint>
+      <controlled-joint>r_shoulder_pan_joint</controlled-joint>
+      <controlled-joint>r_upper_arm_roll_joint</controlled-joint>
+      <controlled-joint>r_elbow_flex_joint</controlled-joint>
+      <controlled-joint>r_forearm_roll_joint</controlled-joint>
+      <controlled-joint>r_wrist_flex_joint</controlled-joint>
+      <controlled-joint>r_wrist_roll_joint</controlled-joint>
+      <controlled-joint>l_shoulder_lift_joint</controlled-joint>
+      <controlled-joint>l_shoulder_pan_joint</controlled-joint>
+      <controlled-joint>l_upper_arm_roll_joint</controlled-joint>
+      <controlled-joint>l_elbow_flex_joint</controlled-joint>
+      <controlled-joint>l_forearm_roll_joint</controlled-joint>
+      <controlled-joint>l_wrist_flex_joint</controlled-joint>
+      <controlled-joint>l_wrist_roll_joint</controlled-joint>
+   </plugin>
   </model>
 </sdf>

File: models/combined-human-pr2-zero-effort/combined-human-pr2.xacro (robot description, xacro)
@@ -11,20 +11,4 @@
    <!-- Human -->
    <xacro:include filename="../human/human.include"/>
-   <plugin name="pr2_arm_controller" filename="libStableControllerPlugin.dylib">
-      <controlled-joint>r_shoulder_lift_joint</controlled-joint>
-      <controlled-joint>r_shoulder_pan_joint</controlled-joint>
-      <controlled-joint>r_upper_arm_roll_joint</controlled-joint>
-      <controlled-joint>r_elbow_flex_joint</controlled-joint>
-      <controlled-joint>r_forearm_roll_joint</controlled-joint>
-      <controlled-joint>r_wrist_flex_joint</controlled-joint>
-      <controlled-joint>r_wrist_roll_joint</controlled-joint>
-      <controlled-joint>l_shoulder_lift_joint</controlled-joint>
-      <controlled-joint>l_shoulder_pan_joint</controlled-joint>
-      <controlled-joint>l_upper_arm_roll_joint</controlled-joint>
-      <controlled-joint>l_elbow_flex_joint</controlled-joint>
-      <controlled-joint>l_forearm_roll_joint</controlled-joint>
-      <controlled-joint>l_wrist_flex_joint</controlled-joint>
-      <controlled-joint>l_wrist_roll_joint</controlled-joint>
-   </plugin>
   </model>
 </sdf>
